File: nref-wifi/nref-wifi.kicad_pcb (KiCad board)
At the start: 2 copper layers, 66 x 32 mm, 8 parts, among them J1 Conn_01x20, J2 Conn_Coaxial_Small

Commit message: add latest PCB updates
Parts:
- removed J2: Conn_Coaxial_Small, Connector_Coaxial:U.FL_Molex_MCRF_73412-0110_Vertical
- removed R1: R_Small, Resistor_SMD:R_0603_1608Metric
- added C1: 10uF, Capacitor_SMD:C_0603_1608Metric, F.Cu at (148.0, 96.0)
- added C2: 10uF, Capacitor_SMD:C_0603_1608Metric, F.Cu at (148.0, 97.5)
- added C3: 10uF, Capacitor_SMD:C_0603_1608Metric, F.Cu at (146.4, 90.8)
- added C4: 10uF, Capacitor_SMD:C_0603_1608Metric, F.Cu at (157.6, 102.4)
- added C5: 10uF, Capacitor_SMD:C_0603_1608Metric, F.Cu at (171.2, 104.4)
- added C6: 10uF, Capacitor_SMD:C_0603_1608Metric, F.Cu at (171.6, 98.6)
- added C7: 0.1uF, Capacitor_SMD:C_0603_1608Metric, F.Cu at (170.3, 108.8)
- added H3: BADGE, footprints:nref-wifi-badge, F.Cu at (179.0, 91.0)
- added R10: 4.75k, Resistor_SMD:R_0603_1608Metric, F.Cu at (166.4, 103.1)
- added R11: 4.75k, Resistor_SMD:R_0603_1608Metric, F.Cu at (167.9, 103.1)
- added R2: 4.75k, Resistor_SMD:R_0603_1608Metric, F.Cu at (143.3, 90.8)
- added R3: 4.75k, Resistor_SMD:R_0603_1608Metric, F.Cu at (144.8, 90.8)
- added R4: 0, Resistor_SMD:R_0603_1608Metric, F.Cu at (169.9, 97.0)
- added R5: 4.75k, Resistor_SMD:R_0603_1608Metric, F.Cu at (167.9, 106.1)
- added R6: 4.75k, Resistor_SMD:R_0603_1608Metric, F.Cu at (166.4, 106.1)
- added R7: 4.75k, Resistor_SMD:R_0603_1608Metric, F.Cu at (156.1, 102.4)
- added R8: 0, Resistor_SMD:R_0603_1608Metric, F.Cu at (168.8, 99.4)
- added R9: 0, Resistor_SMD:R_0603_1608Metric, F.Cu at (170.3, 110.3)
- added U1: TLV75718PDBV, Package_TO_SOT_SMD:SOT-23-5, F.Cu at (171.4, 101.5)
- added X1: ECS-327MVATX-2-CN-TR3, Oscillator:Oscillator_SMD_ECS_2520MV-xxx-xx-4Pin_2.5x2.0mm, F.Cu at (167.2, 109.5)
- moved MOD1 17.0 mm to (156.4, 89.7), turned to 0 degrees
- moved J1 15.3 mm to (156.5, 108.0)
- moved FB1 7.87 mm to (159.2, 101.4), turned to 90 degrees
- moved FB2 7.31 mm to (149.5, 103.2)
Connections:
- FB2 pad 2: Net-(FB2-Pad2) -> 3V3_F
- MOD1 pad 17: Net-(MOD1-VBAT-Pad17) -> 3V3_F
- MOD1 pad 18: Net-(MOD1-VBAT-Pad17) -> 3V3_F
- MOD1 pad 26: unconnected-(MOD1-USB2_RREF-Pad26) -> Net-(MOD1-USB2_RREF)
- MOD1 pad 30: unconnected-(MOD1-VDDIO-Pad30) -> Net-(MOD1-VDDIO)
- MOD1 pad 34: unconnected-(MOD1-SUSCLK-Pad34) -> Net-(MOD1-SUSCLK)
- MOD1 pad 4: unconnected-(MOD1-STRAP_2-Pad4) -> Net-(MOD1-STRAP_2)
- MOD1 pad 44: RK_UART1_CTS_1V8 -> RK_UART1_RTS_1V8
- MOD1 pad 46: RK_UART1_RTS_1V8 -> RK_UART1_CTS_1V8
- MOD1 pad 5: unconnected-(MOD1-STRAP_0-Pad5) -> Net-(MOD1-STRAP_0)
- MOD1 pad 50: Net-(J2-In) -> unconnected-(MOD1-RF_OUT-Pad50)
- MOD1 pad 7: unconnected-(MOD1-VDDIO_RF-Pad7) -> 3V3_F
Routing:
- net +3V3: track 0.00 -> 62.8 mm, vias 0 -> 3
- net GND: track 0.00 -> 61.8 mm, vias 0 -> 67
- net SDIO_D0: track 0.00 -> 41.2 mm, vias 0 -> 2
- net SDIO_D1: track 0.00 -> 38.1 mm, vias 0 -> 2
- net SDIO_D3: track 0.00 -> 35.8 mm, vias 0 -> 2
- net SDIO_CMD: track 0.00 -> 32.5 mm, vias 0 -> 2
- net RK_WIFI_GPIO2: track 0.00 -> 29.1 mm, vias 0 -> 3
- net SDIO_D2: track 0.00 -> 28.9 mm, vias 0 -> 2
- net SDIO_CLK: track 0.00 -> 28.8 mm, vias 0 -> 2
- net RK_UART1_RTS_1V8: track 0.00 -> 26.2 mm, vias 0 -> 2
- net RK_UART1_CTS_1V8: track 0.00 -> 25.5 mm, vias 0 -> 2
- net RK_WIFI_GPIO1: track 0.00 -> 25.0 mm, vias 0 -> 3
- net RK_UART1_TX_1V8: track 0.00 -> 24.9 mm, vias 0 -> 2
- net RK_UART1_RX_1V8: track 0.00 -> 23.2 mm, vias 0 -> 2
- net 3V3_F: track 0.00 -> 23.1 mm
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- added copper zone on B.Cu, net GND
- added copper zone on F.Cu, net GND
Other:
- board size 66 x 32 mm -> 66 x 33 mm
