File: nref-wifi/nref-wifi.kicad_sch (KiCad schematic)
At the start: 8 parts, among them J1 Conn_01x20, J2 Conn_Coaxial_Small

Commit message: add latest PCB updates
Parts:
- removed J2: Conn_Coaxial_Small, Connector_Coaxial:U.FL_Molex_MCRF_73412-0110_Vertical, symbol Connector:Conn_Coaxial_Small
- removed R1: R_Small, Resistor_SMD:R_0603_1608Metric, symbol Device:R_Small
- added C1, C2, C3, C4, C5, C6: 10uF, Capacitor_SMD:C_0603_1608Metric, symbol Device:C_Small
- added C7: 0.1uF, Capacitor_SMD:C_0603_1608Metric, symbol Device:C_Small
- added H3: BADGE, footprints:nref-wifi-badge, symbol Mechanical:MountingHole
- added R10, R11, R2, R3, R5, R6, R7: 4.75k, Resistor_SMD:R_0603_1608Metric, symbol Device:R_Small
- added R4, R8, R9: 0, Resistor_SMD:R_0603_1608Metric, symbol Device:R_Small
- added U1: TLV75718PDBV, Package_TO_SOT_SMD:SOT-23-5, symbol Regulator_Linear:TLV75718PDBV
- added X1: ECS-327MVATX-2-CN-TR3, Oscillator:Oscillator_SMD_ECS_2520MV-xxx-xx-4Pin_2.5x2.0mm, symbol Oscillator:ECS-2520MV-xxx-xx
- FB1, FB2: Manufacturer (none) -> Murata; Manufacturer_No (none) -> BLM18KG221SH1D
- H1, H2: now not fitted
- MOD1: Manufacturer_No (none) -> 453-00046C; Mounting SMT -> (none); Substitutes Allowed NO -> (none)
Connections:
- net +3V3: now also C5.1, R10.2, R11.2, R8.1, R9.2, U1.1 (IN), U1.3 (EN)
- net GND: now also C1.2, C2.2, C3.2, C4.2, C5.2, C6.2, C7.2, R2.1, R3.1, R5.1, R6.1, R7.1, U1.2 (GND), X1.2 (GND)
- net RK_UART1_CTS_1V8: now also MOD1.46 (BT_UART_RTSn); no longer MOD1.44 (BT_UART_CTSn)
- net RK_UART1_RTS_1V8: now also MOD1.44 (BT_UART_CTSn); no longer MOD1.46 (BT_UART_RTSn)
- net RK_WIFI_GPIO1: now also R10.1, R6.2
- net RK_WIFI_GPIO2: now also R11.1, R5.2
- net 3V3_F: now reaches MOD1.17 (VBAT), MOD1.18 (VBAT)
- net 3V3_F: now also FB2.2, MOD1.7 (VDDIO_RF), C1.1, C2.1, C3.1
- net at MOD1.26 (USB2_RREF): now also R7.2
- net at FB1.2, MOD1.28 (USB2_AVDD33): now also C4.1
- net at MOD1.30 (VDDIO): now also R4.2, R8.2
- net at MOD1.34 (SUSCLK): now also X1.3 (OUT)
- net at MOD1.4 (STRAP_2): now also R2.2
- net at MOD1.5 (STRAP_0): now also R3.2
- new net: C7.1, R9.1, X1.1 (Tri-State), X1.4 (VDD)
- new net +1V8: C6.1, R4.1, U1.5 (OUT)
- no-connect marks 11 -> 17
Other:
- note added: "Straps[2-0]: WLAN/BT 000 = USB/USB 101 = SDIO1V8/UART 100 = SDIO3V3/UART"
- note added: "TODO: better harmonics with 3.6V?"
- moved on the sheet: FB1, FB2, J1, MOD1
