File: nref-motherboard/nref-motherboard.kicad_sch (KiCad schematic)
At the start: 250 parts, among them J1 PWR, J10 1-2199230-6, J10 DISP, J11 BAT1, J12 BAT2, J13 SYSCTL_USB, J14 USB_INT2, J16 Conn_01x10_Pin, J17 Conn_01x10_Pin, J17 POWSW, J18 Conn_01x20, J19 SER, J2 Conn_01x12_Pin, J3 10102166A812A, J5 SYSCTL, J6 USB_INT1, J8 Conn_01x12_Pin, J9 Conn_01x14_Pin, Q1 NTMFD6H840NL, Q2 NTMFD6H840NL, SW2 SYS_RESET, SW4 SW_DIP_x08, U1 reform2-som-connector, U10 BQ25756RRVR, U10 W25Q32JVSS, U11 LM62460, U12 TS3USB30EDGSR, U13 TLV75712PDBV, U14 TLV75718PDBV, U2 MAX1837EUT33+T, U26 74HC573, U4 Si52112-B5, U5 LM62460, U6 PCF8523T, U7 USB2514B_Bi, U8 RP2040, Y2 12MHz 18pF, Y2 24MHz, Y3 25MHz, Y4 32.768 kHz

Commit message: add bq25792 charger to schematic
Parts:
- added C100, C101, C103: 47nF, Capacitor_SMD:C_0402_1005Metric, symbol Device:C_Small
- added C102: 4.7uF, symbol Device:C_Small
- added C104, C106, C109: 470nF, Capacitor_SMD:C_0402_1005Metric, symbol Device:C_Small
- added C105, C107, C108, C110, C111, C112, C113, C114, C115, C116: 10uF, Capacitor_SMD:C_0603_1608Metric, symbol Device:C_Small
- added C98, C99: 2.2uF/60V, Capacitor_SMD:C_1206_3216Metric, symbol Device:C_Small
- added D14: Red, LED_SMD:LED_0603_1608Metric, symbol Device:LED_Small
- added L4: 2.2uH, Automated:L_YJYCOIN_YSPIT0660A-XXX, symbol Device:L_Ferrite
- added Q3, Q4, Q5, Q6: Q_NMOS_DGS, symbol Device:Q_NMOS_DGS
- added R85, R86: 2, Resistor_SMD:R_0603_1608Metric, symbol Device:R_Small
- added R87: 2.2k, Capacitor_SMD:C_0603_1608Metric, symbol Device:R_Small
- added R88: 27k, Capacitor_SMD:C_0603_1608Metric, symbol Device:R_Small
- added R89: 100, Capacitor_SMD:C_0603_1608Metric, symbol Device:R_Small
- added R90, R91, R92: 10k, Resistor_SMD:R_0402_1005Metric, symbol Device:R_Small
- added R93: 127k, Capacitor_SMD:C_0603_1608Metric, symbol Device:R_Small
- added R94: 100k, Capacitor_SMD:C_0603_1608Metric, symbol Device:R_Small
- added U15: BQ25792, Automated:Texas_VQFN-HR_RQM_4x4mm_P0.40-0.45mm, symbol meansOfCircuitDesign:BQ25792
- renumbered C109 to C1, C11 to C10, C14 to C12, C22 to C18, C24 to C19, C25 to C20, C26 to C21, C27 to C22, C28 to C23, C29 to C24, C30 to C25, C31 to C26, C32 to C27, C33 to C28, C34 to C29, C4 to C3, C35 to C30, C36 to C31, C40 to C32, C58 to C33, C59 to C34, C60 to C35, C61 to C36, C124 to C37, C126 to C38, C7 to C5, D4 to D1, D10 to D5, D23 to D6, D2 to D7, FB4 to FB1, FB1 to FB2, H5 to H1, J17 to J1, J10 to J4, J1 to J7, L3 to L2, R42 to R1, R46 to R13, R72 to R14, R6 to R17, R43 to R2, R9 to R20, R15 to R23, R16 to R24, R35 to R27, R36 to R28, R38 to R29, R30 to R3, R47 to R32, R48 to R33, R56 to R36, R57 to R37, R58 to R38, R59 to R39, R60 to R40, R61 to R41, R198 to R43, R199 to R44, R110 to R51, R11 to R6, U26 to U2, U2 to U3, U10 to U9, Y2 to Y1
Connections:
- net BAT2_V+ is gone; now on net BAT1_V+: J12.2 (Pin_2), J12.6 (Pin_6), R63.2
- net BAT1_V+: now also R89.1, U15.22 (BAT), U15.23 (BAT)
- net CHRG_ALERT: now also R90.1
- net GND: now also C102.2, C103.1, C104.1, C105.2, C106.1, C107.2, C108.2, C109.1, C110.2, C111.2, C112.2, C113.2, C114.2, C115.2, C116.2, C98.2, C99.2, R88.2, R94.2, U15.27 (GND)
- net REGN: now also C102.1, D14.2 (A), R93.1, U15.5 (REGN)
- net RP_SCL0: now also R91.1
- net RP_SDA0: now also R92.1
- net VCC: now also C109.2, C111.1, C113.1, C114.1, C115.1, C116.1, U15.25 (SYS)
- net VPD: now also Q3.1 (D), R85.1, U15.9 (VAC1)
- net ~{CHRG_CE}: now also U15.13 (~{CE})
- new net: C99.1, R86.2
- new net: R87.1, U15.1 (STAT)
- new net: R91.2, U15.14 (SCL)
- new net: R92.2, U15.15 (SDA)
- new net: R93.2, R94.1, U15.17 (ILIM_HIZ)
- new net: C101.2, U15.19 (BTST2)
- new net: R88.1, U15.20 (PROG)
- new net: R90.2, U15.21 (~{INT})
- new net: C101.1, L4.1, U15.26 (SW2)
- new net: C100.1, L4.2, U15.28 (SW1)
- new net: C106.2, C108.1, C110.1, C112.1, U15.29 (PMID)
- new net: C100.2, U15.4 (BTST1)
- new net: Q3.3 (S), Q5.3 (S)
- new net: D14.1 (K), R87.2
- new net: C98.1, R85.2
- new net: Q4.3 (S), Q6.3 (S)
- new net ACDRV1: Q3.2 (G), Q5.2 (G), U15.11 (ACDRV1)
- new net ACDRV2: Q4.2 (G), Q6.2 (G), U15.10 (ACDRV2)
- new net BATP: C103.2, R89.2, U15.18 (BATP)
- new net D+: U15.6 (D+)
- new net D-: U15.7 (D-)
- new net VBUSp: C104.2, C105.1, C107.1, Q5.1 (D), Q6.1 (D), U15.2 (VBUSp), U15.3 (VBUSp)
- new net V_{IN2}: Q4.1 (D), R86.1, U15.8 (VAC2)
- new net ~{QON}: U15.12 (~{QON})
- no-connect marks 120 -> 121
Other:
- note added: "<-- need to grab footprint from EasyEDA"
- note added: "Consider: - Vishay SISF06DN-T1-GE3 PowerPAK1212-8SCD 68 cent/pair LCSC# C3279460 (30-V dual nMOS 6mOhm each) - AGMSEMI AGM406MNA PDFN-8(5x6) 22 cent/pair LCSC# C5447812 (40-V dual nMOS 10mOhm Rds @4.5Vgs) - GOFORD GT095N04D3 DFN3x3-8L 8.3 cent/each LCSC# C7465423 (40-V single nMOS 7.6mOhm typ Rds @4.5Vgs) - AGMSEMI AGM614MBP PDFN3.3x3.3 23.4 cent/pair LCSC# C7466523 (60-V dual nMOS 20mOhm typ Rds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"
- note added: "New Main/Charge Buck Boost"
- note added: "PROG set for 750 kHz 4S configuration can be overridden over I²C when needed"
- note added: "TODO optional second input"
- note added: "TODO: USB yes, no?"
- note added: "TODO: ship mode/reset"
- note added: "TODO: there's no hardware configuration for LFP/LiPo, needs to be done via I²C on the MCU"
- note added: "around 50uF nominal capacitance should be on Vsys unclear whether it should be per bq25792 or total"
- note added: "can we just connect Vsys pins together? is that OK for the chip?"
- note added: "do not leave floating"
