File: nref-motherboard/nref-motherboard.kicad_sch (KiCad schematic)
At the start: 260 parts, among them J1 POWSW, J10 DISP, J11 BAT1, J12 BAT2, J13 SYSCTL_USB, J14 USB_INT2, J15 SM03B-SRSS-TB, J16 Conn_01x10_Pin, J17 Conn_01x10_Pin, J18 Conn_01x20, J19 SER, J2 Conn_01x12_Pin, J20 Conn_01x20, J3 10102166A812A, J4 1-2199230-6, J5 SYSCTL, J6 USB_INT1, J7 PWR, J8 Conn_01x12_Pin, J9 Conn_01x14_Pin, SW2 SYS_RESET, SW4 SW_DIP_x08, U1 reform2-som-connector, U10 RP2350_60QFN, U11 LM62460, U12 TS3USB30EDGSR, U13 TLV75712PDBV, U14 TLV75718PDBV, U15 BQ25792, U3 MAX1837EUT33+T, U4 Si52112-B5, U5 LM62460, U6 PCF8523T, U7 USB2514B_Bi, U8 PCA9536DP, U9 W25Q128JVS, Y1 12MHz 10pF, Y2 24MHz, Y3 25MHz, Y4 32.768 kHz

Commit message: motherboard: snapshot before d4
Other:
- note added: "TODO: J11+J12: hotplug diodes on V+"
- note added: "TODO: tie ACDRV1+2 to GND!"
Changed lines of the file:
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@@
+		)
+	)
+	(text "TODO: tie ACDRV1+2 to GND!"
+		(exclude_from_sim no)
+		(at 364.49 457.2 0)
+		(effects
+			(font
+				(size 1.27 1.27)
+			)
 		)
 	)
@@
 		)
 	)
+	(text "TODO: J11+J12: hotplug diodes on V+"
+		(exclude_from_sim no)
+		(at 182.88 623.57 0)
+		(effects
+			(font
+				(size 1.27 1.27)
+			)
+		)
+	)

Commit message: motherboard: WIP some TVS, more notes
Parts:
- added D5, D8: ESDS314, Package_TO_SOT_SMD:SOT-23-5, symbol Power_Protection:ESDS304
- R17, R25: value 100k -> 10k
Connections:
- net BAT1_ALERT: now also D5.1 (K)
- net BAT2_ALERT: now also D8.1 (K)
- net GND: now also D5.2 (A), D8.2 (A)
- net at J12.4 (Pin_4), R45.1: now also D8.3 (K)
- net at J12.5 (Pin_5), R46.1: now also D8.4 (K)
- net at J11.4 (Pin_4), R47.1: now also D5.3 (K)
- net at J11.5 (Pin_5), R48.1: now also D5.4 (K)
- no-connect marks 102 -> 104
Other:
- note added: "TODO: Polyfuses?"
- note added: "TODO: TVS"
- note added: "TODO: TVS for pcie?!"
- note added: "TODO: get rid of ferrites, put TVS"
- note added: "TODO: remove FB"
- note removed: "Polyfuses?"
- note removed: "TODO: invert in code"
- note removed: "TODO: protection diodes"
- note removed: "TODO: protection diodes, also on ALERT"
- note removed: "TODO: replace with 100ohms"
- note removed: "check: ESDS314, ESD351, TPD4E1B06"
- moved on the sheet: J12, R45, R46, R47, R48

Commit message: WIP mb v4 re-routing snapshot
Parts:
- removed C33: 10nF, Capacitor_SMD:C_0603_1608Metric, symbol Device:C_Small
- removed C34, C35, C36: 0.1uF, Capacitor_SMD:C_0402_1005Metric, symbol Device:C_Small
- removed FB1, FB3: 100@100MHz 3A, Inductor_SMD:L_0603_1608Metric, symbol pocket-reform-motherboard-rescue:Ferrite_Bead_Small-Device
- added C43: 47uF, Capacitor_SMD:C_0603_1608Metric, symbol Device:C_Small
- C41: footprint Capacitor_SMD:C_0402_1005Metric -> Capacitor_SMD:C_0603_1608Metric
Connections:
- net +3V3: now also C37.1, C38.1, C92.1, J3.4, J4.12, J4.14, J4.16, J4.18, J4.2, J4.4, J4.70, J4.72, J4.74, R51.1, C43.1
- net GND: now also C43.2

Commit message: mb v4: WIP routing snapshot, 39 left
Parts:
- removed FB2, FB4: 220@100MHz 1.4A, Inductor_SMD:L_0603_1608Metric, symbol Device:FerriteBead_Small
Connections:
- net +5V: now also C39.1, C97.1, J14.1 (Pin_1), J6.1 (Pin_1)
- net at J11.4 (Pin_4), R47.1: now also D5.4 (K); no longer D5.3 (K)
- net at J11.5 (Pin_5), R48.1: now also D5.3 (K); no longer D5.4 (K)
Changed lines of the file:
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@@
 	)
 	(junction
+		(at 146.05 647.7)
+		(diameter 0)
+		(color 0 0 0 0)
+	)
+	(junction
 		(at 436.88 207.01)
 		(diameter 0)
@@
 	)
 	(junction
-		(at 614.68 328.93)
+		(at 148.59 645.16)
 		(diameter 0)
 		(color 0 0 0 0)
 	)
 	(junction
-		(at 781.05 532.13)
+		(at 614.68 328.93)
 		(diameter 0)
 		(color 0 0 0 0)
 	)
 	(junction
-		(at 1087.12 139.7)
+		(at 781.05 532.13)
 		(diameter 0)
 		(color 0 0 0 0)
 	)
 	(junction
-		(at 146.05 645.16)
+		(at 1087.12 139.7)
 		(diameter 0)
 		(color 0 0 0 0)
@@
 	)
 	(junction
-		(at 148.59 647.7)
-		(diameter 0)
-		(color 0 0 0 0)
-	)
-	(junction
 		(at 378.46 403.86)
 		(diameter 0)
@@
 	(wire
 		(pts
+			(xy 146.05 647.7) (xy 146.05 651.51)
+		)
+		(stroke
+			(width 0)
+			(type default)
+		)
+	)
+	(wire
+		(pts
 			(xy 627.38 396.24) (xy 636.27 396.24)
 		)
@@
 	(wire
 		(pts
-			(xy 146.05 645.16) (xy 146.05 651.51)
-		)
-		(stroke
-			(width 0)
-			(type default)
-		)
-	)
-	(wire
-		(pts
 			(xy 254 645.16) (xy 266.7 645.16)
 		)
@@
 	(wire
 		(pts
-			(xy 146.05 645.16) (xy 154.94 645.16)
-		)
-		(stroke
-			(width 0)
-			(type default)
-		)
-	)
-	(wire
-		(pts
 			(xy 132.08 590.55) (xy 137.16 590.55)
 		)
@@
 	(wire
 		(pts
-			(xy 1098.55 445.77) (xy 1106.17 445.77)
-		)
-		(stroke
-			(width 0)
-			(type default)
-		)
-	)
-	(wire
-		(pts
 			(xy 707.39 591.82) (xy 707.39 603.25)
 		)
@@
 	(wire
 		(pts
-			(xy 1097.28 483.87) (xy 1104.9 483.87)
-		)
-		(stroke
-			(width 0)
-			(type default)
-		)
-	)
-	(wire
-		(pts
 			(xy 457.2 544.83) (xy 459.74 544.83)
 		)
@@
 	(wire
 		(pts
+			(xy 148.59 645.16) (xy 154.94 645.16)
+		)
+		(stroke
+			(width 0)
+			(type default)
+		)
+	)
+	(wire
+		(pts
 			(xy 707.39 585.47) (xy 758.19 585.47)
 		)
@@
 	(wire
 		(pts
-			(xy 116.84 645.16) (xy 146.05 645.16)
+			(xy 116.84 645.16) (xy 148.59 645.16)
 		)
 		(stroke
@@
 	(wire
 		(pts
+			(xy 146.05 647.7) (xy 160.02 647.7)
+		)
+		(stroke
+			(width 0)
+			(type default)
+		)
+	)
+	(wire
+		(pts
 			(xy 427.99 431.8) (xy 427.99 433.07)
 		)
@@
 	(wire
 		(pts
-			(xy 1071.88 483.87) (xy 1092.2 483.87)
+			(xy 1071.88 483.87) (xy 1104.9 483.87)
 		)
 		(stroke
@@
 	(wire
 		(pts
-			(xy 1073.15 445.77) (xy 1093.47 445.77)
+			(xy 1073.15 445.77) (xy 1106.17 445.77)
 		)
 		(stroke
@@
 	(wire
 		(pts
-			(xy 116.84 647.7) (xy 148.59 647.7)
+			(xy 116.84 647.7) (xy 146.05 647.7)
 		)
 		(stroke
@@
 	(wire
 		(pts
+			(xy 148.59 645.16) (xy 148.59 651.51)
+		)
+		(stroke
+			(width 0)
+			(type default)
+		)
+	)
+	(wire
+		(pts
 			(xy 425.45 408.94) (xy 464.82 408.94)
 		)
@@
 	(wire
 		(pts
-			(xy 148.59 647.7) (xy 160.02 647.7)
-		)
-		(stroke
-			(width 0)
-			(type default)
-		)
-	)
-	(wire
-		(pts
 			(xy 750.57 290.83) (xy 750.57 289.56)
 		)
@@
 	(wire
 		(pts
-			(xy 148.59 647.7) (xy 148.59 651.51)
-		)
-		(stroke
-			(width 0)
-			(type default)
-		)
-	)
-	(wire
-		(pts
 			(xy 147.32 524.51) (xy 185.42 524.51)
 		)
@@
 	)
 	(symbol
-		(lib_id "Device:FerriteBead_Small")
-		(at 1094.74 483.87 270)
-		(unit 1)
-		(exclude_from_sim no)
-		(in_bom yes)
-		(on_board yes)
-		(dnp no)
-		(property "Reference" "FB4"
-			(at 1095.9084 486.41 0)
-			(effects
-				(font
-					(size 1.27 1.27)
-				)
-				(justify left)
-			)
-		)
-		(property "Value" "220@100MHz 1.4A"
-			(at 1093.597 486.41 0)
-			(effects
-				(font
-					(size 1.27 1.27)
-				)
-				(justify left)
-			)
-		)
-		(property "Footprint" "Inductor_SMD:L_0603_1608Metric"
-			(at 1094.74 482.092 90)
-			(effects
-				(font
-					(size 1.27 1.27)
-				)
-				(hide yes)
-			)
-		)
-		(property "Datasheet" "~"
-			(at 1094.74 483.87 0)
-			(effects
-				(font
-					(size 1.27 1.27)
-				)
-				(hide yes)
-			)
-		)
-		(property "Description" ""
-			(at 1094.74 483.87 0)
-			(effects
-				(font
-					(size 1.27 1.27)
-				)
-				(hide yes)
-			)
-		)
-		(property "Manufacturer_No" "BLM18KG221SN1D"
-			(at 1094.74 483.87 0)
-			(effects
-				(font
-					(size 1.27 1.27)
-				)
-				(hide yes)
-			)
-		)
-		(property "Manufacturer" "Murata"
-			(at 1094.74 483.87 0)
-			(effects
-				(font
-					(size 1.27 1.27)
-				)
-				(hide yes)
-			)
-		)
-		(property "LCSC" "C88980"
-			(at 1094.74 483.87 0)
-			(effects
-				(font
-					(size 1.27 1.27)
-				)
-				(hide yes)
-			)
-		)
-		(pin "1"
-		)
-		(pin "2"
-		)
-		(instances
-			(project "nref-motherboard"
-				(path "/a432b2af-5748-42a5-94fe-8be4ed1e5510"
-					(reference "FB4")
-					(unit 1)
-				)
-			)
-		)
-	)
-	(symbol
 		(lib_id "Device:C_Small")
 		(at 412.75 453.39 180)
@@
 					(unit 1)
 				)
-			)
-		)
-	)
-	(symbol
-		(lib_id "Device:FerriteBead_Small")
-		(at 1096.01 445.77 270)
-		(unit 1)
-		(exclude_from_sim no)
-		(in_bom yes)
-		(on_board yes)
-		(dnp no)
-		(property "Reference" "FB2"
-			(at 1097.1784 448.31 0)
-			(effects
-				(font
-					(size 1.27 1.27)
-				)
-				(justify left)
-			)
-		)
-		(property "Value" "220@100MHz 1.4A"
-			(at 1094.867 448.31 0)
-			(effects
-				(font
-					(size 1.27 1.27)
-				)
-				(justify left)
-			)
-		)
-		(property "Footprint" "Inductor_SMD:L_0603_1608Metric"
-			(at 1096.01 443.992 90)
-			(effects
-				(font
-					(size 1.27 1.27)
-				)
-				(hide yes)
-			)
-		)
-		(property "Datasheet" "~"
-			(at 1096.01 445.77 0)
-			(effects
-				(font
-					(size 1.27 1.27)
-				)
-				(hide yes)
-			)
-		)
-		(property "Description" ""
-			(at 1096.01 445.77 0)
-			(effects
-				(font
-					(size 1.27 1.27)
-				)
-				(hide yes)
-			)
-		)
-		(property "Manufacturer_No" "BLM18KG221SN1D"
-			(at 1096.01 445.77 0)
-			(effects
-				(font
-					(size 1.27 1.27)
-				)
-				(hide yes)
-			)
-		)
-		(property "Manufacturer" "Murata"
-			(at 1096.01 445.77 0)
-			(effects
-				(font
-					(size 1.27 1.27)
-				)
-				(hide yes)
-			)
-		)
-		(property "LCSC" "C88980"
-			(at 1096.01 445.77 0)
-			(effects
-				(font
-					(size 1.27 1.27)
-				)
-				(hide yes)
-			)
-		)
-		(pin "1"
-		)
-		(pin "2"
-		)
-		(instances
-			(project "pocket-reform-motherboard"
-				(path "/63c56ea4-91a3-4172-b9de-a4388cc8f894"
-					(reference "FB1")
-					(unit 1)
-				)
-			)
-			(project "nref-motherboard"
-				(path "/a432b2af-5748-42a5-94fe-8be4ed1e5510"
-					(reference "FB2")
-					(unit 1)
-				)

Commit message: WIP D-4 fully routed, still needs polishing
Parts:
- added H8: NGFF-Mount, footprints:WA-SMSI-M2, symbol Mechanical:MountingHole_Pad
Connections:
- net +3V3: now also J19.1 (Pin_1)
- net GND: now also H8.1
- net STANDBY_3V3: no longer J13.1 (Pin_1), J19.1 (Pin_1)
- no-connect marks 104 -> 105
Other:
- note added: "NOTE: there's no hardware configuration for LFP/LiPo, needs to be done via I²C on the MCU"
- note added: "NOTE: these pulldowns were not strong enough, 10k works in practice"
- note removed: "SDA1 latched up"
- note removed: "TODO: get rid of ferrites, put TVS"
- note removed: "TODO: protect these!"
- note removed: "TODO: protection, this chip died"
- note removed: "TODO: remove FB"
- note removed: "TODO: there's no hardware configuration for LFP/LiPo, needs to be done via I²C on the MCU"
- note removed: "TODO: these pulldowns are not strong enough, 10k works in practice"
- note removed: "TODO: very dangerous!"
- note removed: "actually, probably rp2350a damaged?"
