File: nref-motherboard/nref-motherboard.kicad_pcb (KiCad board)
At the start: 6 copper layers, 122.6 x 75.6 mm, 257 parts, among them J1 POWSW, J10 DISP, J11 BAT1, J12 BAT2, J13 SYSCTL_USB, J14 USB_INT2, J15 SM03B-SRSS-TB, J16 Conn_01x10_Pin, J17 Conn_01x10_Pin, J18 Conn_01x20, J19 SER, J2 Conn_01x12_Pin, J20 Conn_01x20, J3 10102166A812A, J4 1-2199230-6, J5 SYSCTL, J6 USB_INT1, J7 PWR, J8 Conn_01x12_Pin, J9 Conn_01x14_Pin, SW2 SYS_RESET, SW4 SW_DIP_x08, U1 reform2-som-connector, U10 RP2350_60QFN, U11 LM62460, U12 TS3USB30EDGSR, U13 TLV75712PDBV, U14 TLV75718PDBV, U15 BQ25792, U3 MAX1837EUT33+T, U4 Si52112-B5, U5 LM62460, U6 PCF8523T, U7 USB2514B_Bi, U8 PCA9536DP, U9 W25Q128JVS, Y1 12MHz 10pF, Y2 24MHz, Y3 25MHz, Y4 32.768 kHz

Commit message: mb: wip
Routing:
- net GND: track 340.0 -> 336.6 mm, vias 268 -> 271
Other:
- board text removed: "TODO: QON pull?"
Changed lines of the file:
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@@
 		)
 	)
-	(gr_text "TODO: QON pull?"
-		(at 83.25 101.95 0)
-		(layer "F.SilkS")
-		(effects
-			(font
-				(size 1.5 1.5)
-				(thickness 0.3)
-				(bold yes)
-			)
-			(justify left bottom)
-		)
-	)
 	(gr_text "PROG"
 		(at 58.6 107.4 90)
@@
 	)
 	(via
-		(at 132.3 109.7)
+		(at 132.25 110.15)
+		(size 0.6)
+		(drill 0.3)
+		(layers "F.Cu" "B.Cu")
+		(net 2)
+	)
+	(via
+		(at 72.6 107.85)
 		(size 0.6)
 		(drill 0.3)
@@
 	)
 	(via
-		(at 112.8 109.6)
+		(at 112.75 110.15)
 		(size 0.6)
 		(drill 0.3)
@@
 	)
 	(via
-		(at 109.8 109.6)
+		(at 109.75 110.15)
 		(size 0.6)
 		(drill 0.3)
@@
 	)
 	(via
-		(at 114.3 109.6)
+		(at 114.25 110.15)
 		(size 0.6)
 		(drill 0.3)
@@
 	)
 	(via
-		(at 111.3 109.6)
+		(at 111.25 110.15)
 		(size 0.6)
 		(drill 0.3)
@@
 	)
 	(via
-		(at 121.5 109.7)
+		(at 121.5 110.15)
 		(size 0.6)
 		(drill 0.3)
@@
 	)
 	(via
+		(at 96 113.95)
+		(size 0.6)
+		(drill 0.3)
+		(layers "F.Cu" "B.Cu")
+		(net 2)
+	)
+	(via
 		(at 47.9 123.1)
 		(size 0.5)
@@
 	)
 	(via
+		(at 71.05 106.95)
+		(size 0.6)
+		(drill 0.3)
+		(layers "F.Cu" "B.Cu")
+		(net 2)
+	)
+	(via
 		(at 58.4 111.2)
 		(size 0.6)
@@
 	)
 	(via
-		(at 133.7 109.7)
+		(at 133.75 110.15)
 		(size 0.6)
 		(drill 0.3)
@@
 	)
 	(via
-		(at 124.5 109.7)
+		(at 124.5 110.15)
 		(size 0.6)
 		(drill 0.3)
@@
 	)
 	(via
-		(at 94.6 111.5)
+		(at 94.75 112.25)
 		(size 0.6)
 		(drill 0.3)
@@
 	)
 	(segment
-		(start 121.5 111.25)
-		(end 121.5 109.7)
-		(width 0.2)
+		(start 60.9 110.6)
+		(end 60.9 109.2)
+		(width 0.3)
 		(layer "B.Cu")
 		(net 2)
 	)
 	(segment
-		(start 109.75 109.65)
-		(end 109.8 109.6)
+		(start 121.5 111.25)
+		(end 121.5 110.15)
 		(width 0.2)
 		(layer "B.Cu")
@@
 	)
 	(segment
-		(start 60.9 110.6)
-		(end 60.9 109.2)
-		(width 0.3)
-		(layer "B.Cu")
-		(net 2)
-	)
-	(segment
 		(start 100.95 114.25)
 		(end 101.8 115.1)
@@
 	)
 	(segment
-		(start 114.25 109.65)
-		(end 114.3 109.6)
-		(width 0.2)
-		(layer "B.Cu")
-		(net 2)
-	)
-	(segment
 		(start 58.4 111.2)
 		(end 60.3 111.2)
@@
 	)
 	(segment
+		(start 111.25 110.15)
+		(end 111.25 111.25)
+		(width 0.2)
+		(layer "B.Cu")
+		(net 2)
+	)
+	(segment
 		(start 87.5 128.65)
 		(end 87 128.15)
@@
 	)
 	(segment
+		(start 94.75 112.25)
+		(end 94.75 111.35)
+		(width 0.2)
+		(layer "B.Cu")
+		(net 2)
+	)
+	(segment
 		(start 50.1 109.2)
 		(end 50.1 107.6)
@@
 	)
 	(segment
+		(start 114.25 110.15)
+		(end 114.25 111.25)
+		(width 0.2)
+		(layer "B.Cu")
+		(net 2)
+	)
+	(segment
 		(start 50.1 107.6)
 		(end 49.6 107.1)
@@
 	)
 	(segment
-		(start 111.25 109.65)
-		(end 111.3 109.6)
-		(width 0.2)
-		(layer "B.Cu")
-		(net 2)
-	)
-	(segment
 		(start 35.5 110.1)
 		(end 35.8 110.4)
@@
 	)
 	(segment
-		(start 133.75 111.25)
-		(end 133.75 109.75)
-		(width 0.2)
-		(layer "B.Cu")
-		(net 2)
-	)
-	(segment
 		(start 56.2 146.8)
 		(end 56.1 146.9)
@@
 	)
 	(segment
-		(start 112.75 111.25)
-		(end 112.75 109.65)
+		(start 132.25 110.15)
+		(end 132.25 111.25)
 		(width 0.2)
 		(layer "B.Cu")
@@
 	)
 	(segment
+		(start 133.75 110.15)
+		(end 133.75 111.25)
+		(width 0.2)
+		(layer "B.Cu")
+		(net 2)
+	)
+	(segment
 		(start 143.8 150)
 		(end 143.1 150.7)
@@
 	)
 	(segment
-		(start 124.5 111.25)
-		(end 124.5 109.7)
-		(width 0.2)
-		(layer "B.Cu")
-		(net 2)
-	)
-	(segment
 		(start 102.45 111.85)
 		(end 103.675 113.075)
@@
 	)
 	(segment
-		(start 94.6 111.5)
-		(end 96 110.1)
-		(width 0.2)
-		(layer "B.Cu")
-		(net 2)
-	)
-	(segment
 		(start 84.4 122.75)
 		(end 84.25 122.9)
@@
 	)
 	(segment
+		(start 124.5 111.25)
+		(end 124.5 110.15)
+		(width 0.2)
+		(layer "B.Cu")
+		(net 2)
+	)
+	(segment
 		(start 99.45 111.25)
 		(end 99.45 110.4)
@@
 	)
 	(segment
-		(start 111.25 111.25)
-		(end 111.25 109.65)
-		(width 0.2)
-		(layer "B.Cu")
-		(net 2)
-	)
-	(segment
 		(start 73.45 137.9)
 		(end 73.45 136.903932)
@@
 	)
 	(segment
-		(start 132.25 109.75)
-		(end 132.3 109.7)
-		(width 0.2)
-		(layer "B.Cu")
-		(net 2)
-	)
-	(segment
 		(start 143.3 124.5)
 		(end 143 124.2)
@@
 	)
 	(segment
-		(start 114.25 111.25)
-		(end 114.25 109.65)
-		(width 0.2)
-		(layer "B.Cu")
-		(net 2)
-	)
-	(segment
 		(start 90.8 114.3)
 		(end 91.975 114.3)
@@
 	)
 	(segment
+		(start 96 110.1)
+		(end 97.5 110.1)
+		(width 0.2)
+		(layer "B.Cu")
+		(net 2)
+	)
+	(segment
 		(start 144.5 124.5)
 		(end 143.3 124.5)
@@
 	)
 	(segment
+		(start 94.75 111.35)
+		(end 96 110.1)
+		(width 0.2)
+		(layer "B.Cu")
+		(net 2)
+	)
+	(segment
 		(start 97.95 110.4)
 		(end 97.65 110.1)
@@
 	)
 	(segment
-		(start 132.25 111.25)
-		(end 132.25 109.75)
-		(width 0.2)
-		(layer "B.Cu")
-		(net 2)
-	)
-	(segment
 		(start 90.4 112.4)
 		(end 90.4 113.9)
@@
 	)
 	(segment
-		(start 96 110.1)
-		(end 97.5 110.1)
+		(start 109.75 110.15)
+		(end 109.75 111.25)
 		(width 0.2)
 		(layer "B.Cu")
@@
 	)
 	(segment
-		(start 112.75 109.65)
-		(end 112.8 109.6)
-		(width 0.2)
-		(layer "B.Cu")
-		(net 2)
-	)
-	(segment
 		(start 43.3 109.2)
 		(end 43.3 107.4)
@@
 	)
 	(segment
-		(start 133.75 109.75)
-		(end 133.7 109.7)
-		(width 0.2)
-		(layer "B.Cu")
-		(net 2)
-	)
-	(segment
 		(start 89.65 126.83)
 		(end 89.18 127.3)
@@
 	)
 	(segment
-		(start 109.75 111.25)
-		(end 109.75 109.65)
-		(width 0.2)
-		(layer "B.Cu")
-		(net 2)
-	)
-	(segment
 		(start 77.55 140.7)
 		(end 77.55 141.1)
@@
 		(width 0.2)
 		(layer "B.Cu")
+		(net 2)
+	)
+	(segment
+		(start 112.75 110.15)
+		(end 112.75 111.25)
+		(width 0.2)
+		(layer "B.Cu")

Commit message: mb: further pcb cleanups
Routing:
- net GND: track 336.6 -> 326.7 mm, vias 271 -> 292
- net Net-(U1-QSPIA_DATA2): track 9.82 -> 10.3 mm
Other:
- board text removed: "TODO: diff pair gnd vias"
- board text removed: "TODO: unify via sizes"
