File: nref-camera/reform-camera.kicad_sch (KiCad schematic)
At the start: 131 parts, among them J2 Conn_01x04, J3 Conn_ARM_JTAG_SWD_10, J4 Conn_01x24, U1 TXS0104EPWRG4, U12 FAN53600AUC28X, U13 CYUSB306X, U14 FAN53611AUC18X, U15 TLV71715P, U16 TPS2290x, U17 TPS2290x, U2 TXS0104EPWRG4, U21 74LVC2G17, U3 AT25FF041A-UUN-T, U4 LM2830XQMFE/NOPB, X1 ECS-1618-240-BN-TR, X2 NZ2520SB-32.768KHZ-NSA3534C, X3 ECS-1618-192-BN-TR

Commit message: camera: redesigned and fully routed
Parts:
- removed C10, C26: 0.1uF, Capacitor_SMD:C_0402_1005Metric, symbol Device:C_Small
- removed C4, C5: 22uF, Capacitor_SMD:C_0603_1608Metric, symbol Device:C_Small
- removed D1: PMEG1020EA,115, Diode_SMD:D_SOD-323, symbol Device:D_Schottky_Small_Filled
- removed J4: Conn_01x24, reform-camera:FPC_24, symbol Connector_Generic:Conn_01x24
- removed L4: 3.3uH, Inductor_SMD:L_1210_3225Metric, symbol Device:L_Small
- removed R10, R9: 10k, Resistor_SMD:R_0402_1005Metric, symbol Device:R_Small
- removed R3: 100k, Resistor_SMD:R_0201_0603Metric, symbol Device:R_Small
- removed R53, R54, R58, R59, R60: 0R, Resistor_SMD:R_0201_0603Metric, symbol Device:R_Small
- removed R6: 1k, Resistor_SMD:R_0402_1005Metric, symbol Device:R_Small
- removed R7: 0, Resistor_SMD:R_0402_1005Metric, symbol Device:R_Small
- removed TP11, TP6, TP7, TP8, TP9: TestPoint, reform-camera:TestPoint_Pad_D0.7mm, symbol Connector:TestPoint
- removed U2: TXS0104EPWRG4, footprints:SOP65P640X120-14N, symbol TXS0104EPWRG4:TXS0104EPWRG4
- removed U4: LM2830XQMFE/NOPB, Package_TO_SOT_SMD:SOT-23-5, symbol pocket-reform:LM2830XQMFE
- added C14: 2.2u, Capacitor_SMD:C_0402_1005Metric, symbol Device:C_Small
- added C15: 4.7u, Capacitor_SMD:C_0402_1005Metric, symbol Device:C_Small
- added J1: Conn_01x12_Pin, Connector_FFC-FPC:Hirose_FH12-12S-0.5SH_1x12-1MP_P0.50mm_Horizontal, symbol Connector:Conn_01x12_Pin
- added J4: Conn_01x20, Connector_JST:JST_SH_SM20B-SRSS-TB_1x20-1MP_P1.00mm_Horizontal, symbol Connector_Generic:Conn_01x20
- added L1: 470nH 1.1A 120mΩ, Inductor_SMD:L_0805_2012Metric, symbol Device:L_Small
- added R14: 10k, Resistor_SMD:R_0402_1005Metric, symbol Device:R_Small
- added R15: 0R, Resistor_SMD:R_0402_1005Metric, symbol Device:R_Small
- added U11: FAN53611AUC12X, reform-camera:WLCSP-6_2x3_0.8x1.2mm, symbol reform-camera:FAN536xx
- C12, C13, C22, C25, C29, C30, C34, C38, C39, C42, C43, C44, C45, C46, C47, C48, C50, C51, C52, C53, C57, C58, C59: footprint Capacitor_SMD:C_0201_0603Metric -> Capacitor_SMD:C_0402_1005Metric
- J2: value Conn_01x04 -> Conn_01x03; footprint Connector_PinSocket_2.54mm:PinSocket_1x04_P2.54mm_Vertical -> Connector_PinSocket_2.54mm:PinSocket_1x03_P2.54mm_Vertical; symbol Connector_Generic:Conn_01x04 -> Connector_Generic:Conn_01x03
- R16, R17, R18, R19, R20, R22, R23, R24, R25, R26, R27, R28, R29, R35, R36, R37, R62, R64: footprint Resistor_SMD:R_0201_0603Metric -> Resistor_SMD:R_0402_1005Metric
- R63: footprint Resistor_SMD:R_0805_2012Metric -> Resistor_SMD:R_0603_1608Metric
- U1: footprint footprints:SOP65P640X120-14N -> reform-camera:SOP65P640X120-14N
Connections:
- net UART_RX is gone; now on net UART_RX_CX3: J2.2 (Pin_2)
- net UART_TX is gone; now on net UART_TX_CX3: J2.3 (Pin_3)
- net +1V2: now also C15.1, L1.2, U11.C1 (FB)
- net CAM_AF_VCC: now also J4.2 (Pin_2)
- net CAM_AVDD: now also J4.18 (Pin_18)
- net CAM_DOVDD: now also J4.11 (Pin_11)
- net CAM_DVDD: now also J4.12 (Pin_12)
- net CAM_MCLK: now also J4.13 (Pin_13)
- net CAM_MIPI_CN: now also J4.6 (Pin_6)
- net CAM_MIPI_CP: now also J4.7 (Pin_7)
- net CAM_MIPI_D0N: now also J4.3 (Pin_3)
- net CAM_MIPI_D0P: now also J4.4 (Pin_4)
- net CAM_MIPI_D1N: now also J4.9 (Pin_9)
- net CAM_MIPI_D1P: now also J4.10 (Pin_10)
- net CAM_PWDNB: now also J4.14 (Pin_14)
- net CAM_RST: now also J4.15 (Pin_15)
- net CAM_SCL: now also J4.16 (Pin_16)
- net CAM_SDA: now also J4.17 (Pin_17)
- net CAM_STROBE: now also J4.20 (Pin_20)
- net GND: now also C14.2, C15.2, J1.12 (Pin_12), J1.3 (Pin_3), J1.6 (Pin_6), J1.9 (Pin_9), J4.1 (Pin_1), J4.5 (Pin_5), J4.8 (Pin_8), R15.1, U11.C2 (GND)
- net GNDA: now also J4.19 (Pin_19)
- net MISO: now also TP4.1
- net USB_D+: now also J1.2 (Pin_2)
- net USB_D-: now also J1.1 (Pin_1)
- net VBUS: now also C14.1, J1.10 (Pin_10), J1.11 (Pin_11), R14.1, U11.A2 (VIN)
- net at R1.2, R4.1, U3.E3 (~{WP}): no longer TP4.1
- net SSRX+ renamed USB_RXP
- net USB_RXP: now also J1.8 (Pin_8)
- net SSRX- renamed USB_RXN
- net USB_RXN: now also J1.7 (Pin_7)
- net SSTX+ renamed USB_TXP
- net USB_TXP: now also J1.5 (Pin_5)
- net SSTX- renamed USB_TXN
- net USB_TXN: now also J1.4 (Pin_4)
- removed net UART_VCC: J2.4 (Pin_4)
- new net: R15.2, U11.A1 (MODE)
- new net: L1.1, U11.B1 (SW)
- new net: R14.2, U11.B2 (EN)
- no-connect marks 15 -> 19
Other:
- note added: "1.8V!"
- note added: "TODO: what about those unconnected pins?"
- note added: "USB3 to host (flipped)"
- note removed: "1A"
- note removed: "=1.2V"
- note removed: "Itentionally Swapped"
- note removed: "TODO: ???"

Commit message: camera: d-3 done, off to board house
Parts:
- removed H4: MountingHole_Pad, MountingHole:MountingHole_2.2mm_M2_Pad, symbol Mechanical:MountingHole_Pad
- removed U15: TLV71715P, Package_DFN_QFN:UDFN-4-1EP_1x1mm_P0.65mm_EP0.48x0.48mm, symbol reform-camera:TLV742P
- added H4: BADGE, reform-camera:nref-camera-badge, symbol Mechanical:MountingHole
- added J5: Conn_01x03, Connector_JST:JST_SH_SM03B-SRSS-TB_1x03-1MP_P1.00mm_Horizontal, symbol Connector_Generic:Conn_01x03
- added J6: USB_INT1, Connector_JST:JST_SH_SM04B-SRSS-TB_1x04-1MP_P1.00mm_Horizontal, symbol Connector:Conn_01x04_Male
- added Q1: AO3416, Package_TO_SOT_SMD:SOT-23, symbol Transistor_FET:AO3400A
- added R3: 20k, Resistor_SMD:R_0402_1005Metric, symbol Device:R_Small
- added R6: 16.9k, Resistor_SMD:R_0402_1005Metric, symbol Device:R_Small
- added R7: 36.5k, Resistor_SMD:R_0402_1005Metric, symbol Device:R_Small
- added R9: 10k, Resistor_SMD:R_0402_1005Metric, symbol Device:R_Small
- added U15: TLV75801PDBV, Package_TO_SOT_SMD:SOT-23-5, symbol Regulator_Linear:TLV75801PDBV
Connections:
- net +2V8: now also U15.1 (IN)
- net CAM_DVDD: now also R3.1, U15.5 (OUT)
- net DVDD_SUPPLY_EN: now also U15.3 (EN)
- net GND: now also J5.1 (Pin_1), J6.4 (Pin_4), Q1.2 (S), R6.2, R9.2, U15.2 (GND)
- net USB_D+: now also J6.3 (Pin_3)
- net USB_D-: now also J6.2 (Pin_2)
- net VBUS: now also J5.3 (Pin_3); no longer J1.10 (Pin_10), J1.11 (Pin_11)
- net DVDD_1V5_SEL: now reaches U13.C8 (GPIO22)
- net DVDD_1V5_SEL: now also Q1.1 (G), R9.1
- new net: R3.2, R6.1, R7.1, U15.4 (FB)
- new net: Q1.3 (D), R7.2
- new net +5V: J1.10 (Pin_10), J1.11 (Pin_11), J5.2 (Pin_2), J6.1 (Pin_1)
- no-connect marks 19 -> 20
Other:
- note added: "1.2V"
- note added: "1.5V"
- note added: "A switch controlling the connection of +5V to VBUS is connected here. GND for powering an LED on the switch board."
- note added: "Alternative USB2"
- note added: "Killswitch"
- note added: "USB2"
- note added: "USB3"
- note added: "optional 1.2V/1.5V DVDD Supply"
- note added: "~11.5k combined"
- note removed: "TODO: unidirectional A->B? pulls?"
- note removed: "TODO: what about those unconnected pins?"
- note removed: "optional 1.5V DVDD Supply"
- moved on the sheet: C18, C19, FB2, H1, H2, H3, R18

Commit message: add latest PCB updates
Parts:
- added H5: MountingHole_Pad, MountingHole:MountingHole_2.2mm_M2_Pad, symbol Mechanical:MountingHole_Pad
- added R10: 0R, Resistor_SMD:R_0402_1005Metric, symbol Device:R_Small
- added R11: 10k, Resistor_SMD:R_0402_1005Metric, symbol Device:R_Small
- C1, C3: MPN (none) -> GRM155R71C104KA88J; Manufacturer Yageo -> Murata; Manufacturer_No CC0402KRX7R7BB104 -> (none)
- C11, C14, C17, C35: value 2.2u -> 2.2uF
- C12, C13, C2, C22, C29, C30, C42, C43, C44, C45, C46, C47, C48, C49, C51, C54, C55, C56, C57, C58, C59, C60: value 0.1u -> 0.1uF; MPN GRM033R61E104KE14D -> GRM155R71C104KA88J
- C15, C20: value 4.7u -> 4.7uF; MPN GRJ155R61A475ME11J -> GRT155C81A475ME13J
- C16, C40, C41: value 10u -> 10uF; MPN (none) -> C0603C106M8PAC7411; Manufacturer (none) -> Kemet
- C18, C19, C23, C24: value 1u -> 1uF
- C21, C36, C37: value 22u -> 22uF; MPN GRT188C80J226ME13D -> MSASJ168BC6226MTNA01; Manufacturer Murata -> Taiyo Yuden
- C25, C34, C38, C39, C50, C52, C53: value 0.01u -> 0.01uF; MPN GRM033R71A103KA01D -> C0402C103K8RAC7411; Manufacturer Murata -> Kemet
- FB2, FB3, FB4, FB5, FB6, FB7, FB8, FB9: MPN (none) -> MI0603L301R-10; Manufacturer (none) -> Laird
- H1, H2, H3, H4, TP1, TP10, TP2, TP3, TP4, TP5: MPN (none) -> DNP; Manufacturer (none) -> DNP
- J1: MPN (none) -> FH12-12S-0.5SH(55); Manufacturer_No FH12-12S-0.5SH(55) -> (none)
- J2: MPN (none) -> DNP; Manufacturer (none) -> DNP; now not fitted
- J3: MPN 62201021121 -> 62201021121 (DNP); now not fitted
- J4: MPN (none) -> SM20B-SRSS-TB; Manufacturer (none) -> JST
- J5: MPN (none) -> SM03B-SRSS-TB; Manufacturer (none) -> JST
- J6: MPN (none) -> SM04B-SRSS-TB; Manufacturer_No SM04B-SRSS-TB -> (none)
- Q1: MPN (none) -> DMN2024U-7; Manufacturer (none) -> Diodes
- R1, R15, R16, R20: MPN ERJ-1GN0R00C -> CRCW04020000Z0EDC; Manufacturer Panasonic -> Vishay
- R14, R18, R19, R23, R27, R33, R34, R64, R9: MPN RC0201DR-0710KL -> RC0402FR-7D10KL
- R17, R25, R26, R28, R29: MPN ERJ-1GN0R00C -> CRCW04020000Z0EDC; Manufacturer Panasonic -> Vishay; now not fitted
- R2: MPN (none) -> CRCW04021K00FKEDC; Manufacturer_No CRCW04021K00FKEDC -> (none)
- R21: MPN RC0402FR-7D1KL -> CRCW04021K00FKEDC; Manufacturer Yageo -> Vishay
- R22, R24: MPN RC0201DR-0710KL -> RC0402FR-7D10KL; now not fitted
- R3: MPN (none) -> RC0402FR-7D20KL; Manufacturer (none) -> Yageo
- R35, R36, R37: MPN RC0201FR-0722RL -> RC0402FR-7D22RL
- R4, R5, R62: MPN RC0201JR-13100KL -> RC0402FR-07100KL
- R6: MPN (none) -> CRCW040216K9FKTD; Manufacturer (none) -> Vishay
- R63: MPN CRCW08050000Z0EAHP -> CRCW060320K0FKEAC; Manufacturer Vishay Dale -> Vishay
- R7: MPN (none) -> RP0402BRD0736K5L; Manufacturer (none) -> Yageo
- R8: MPN CR0402-FX-4701GLF -> RC0402FR-074K7L; Manufacturer Bourns -> Yageo
- U1: MPN (none) -> TXS0104EPWRG4; Manufacturer_No TXS0104EPWRG4 -> (none)
- U15: MPN (none) -> TLV75801PDBV; Manufacturer (none) -> Texas Instruments
Connections:
- net +5V: now also R10.2
- net GND: now also H5.1, R11.2
- net USB_RXN: now also J1.4 (Pin_4); no longer J1.7 (Pin_7)
- net USB_RXP: now also J1.5 (Pin_5); no longer J1.8 (Pin_8)
- net USB_TXN: now also J1.7 (Pin_7); no longer J1.4 (Pin_4)
- net USB_TXP: now also J1.8 (Pin_8); no longer J1.5 (Pin_5)
- net VBUS: now also R10.1
- net at R17.2, TP5.1, U13.H6 (MIPI_RESET): now also R11.1
Other:
- note added: "For Testing Only"
- note added: "RX/TX crossed vs D-1"
- note added: "added in D-2"
- moved on the sheet: H4

Commit message: snapshot before merge
Parts:
- X1: value ECS-1618-240-BN-TR -> ECS-1618-240-BN-TR
- X3: value ECS-1618-192-BN-TR -> ECS-1618-192-BN-TR

Commit message: add various notes in schematics
Other:
- note added: "TODO: ESD"
Changed lines of the file:
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@@
 		)
 	)
+	(text "TODO: ESD"
+		(exclude_from_sim no)
+		(at 90.17 255.27 0)
+		(effects
+			(font
+				(size 1.27 1.27)
+			)
+		)
+	)
 	(text "USB2"
 		(exclude_from_sim no)
@@
 			"AAAAAAAAAAAAAAAAAAAAAAAAAAAAAAAAAAAAAAAAAAAAAAAAAAAAAAAAAAAAAAAAAAAAAAAAAAAA"
 			"AAAAAAAAAAAAAAAAAAAAAAAAAAAAAAAAAAAAAAAAAAAAAAAAAAAAAAAAAAAAAAAAAAAAAAAAAAAA"
-			"AAAAAAAAAAAAAAAAAAAAAAAAAAAAAAAAAADoXXQL82V9VvNkf4/xZA=="
+			"AAAAAAAAAAAAAAAAAAAAAAAAAAAAAAAAAADoXXQL82V9VvNkf4/xZAAAAAAAAAAAAAAAAAAAAAAA"
+			"AAAAAAAAAAAAAAAAAAAAAAAAAAAAAAAAAAAAAAAAAAAAAAAAAAAAAAAAAAAAAAAAAAAAAAAAAAAA"
+			"AAAAAAAAAAAAAAAAAAAAAAAAAAAAAAAAAAAAAAAAAAAAAAAAAAAAAAAAAAAAAAAAAAAAAAAAAAAA"
+			"AAAAAAAAAAAAAAAAAAAAAAAAAAAAAAAAAAAAAAAAAAAAAAAAAAAAAAAAAAAAAAAAAAAAAAAAAAAA"
+			"AAAAAAAAAAAAAAAAAAAAAAAAAAAAAAAAAAAAAAAAAAAAAAAAAAAAAAAAAAAAAAAAAAAAAAAAAAAA"
+			"AAAAAAAAAAAAAAAAAAAAAAAAAAAAAAAAAAAAAAAAAAAAAAAAAAAAAAAAAAAAAAAAAAAAAAAAAAAA"
+			"AAAAAAAAAAAAAAAAAAAAAAAAAAAAAAAAAAAAAAAAAAAAAAAAAAAAAAAAAAAAAAAAAAAAAAAAAAAA"
+			"AAAAAAAAAAAAAAAAAAAAAAAAAAAAAAAAAAAAAAAAAAAAAAAAAAAAAAAAAAAAAAAAAAAAAAAAAAAA"
+			"AAAAAAAAAAAAAAAAAAAAAAAAAAAAAAAAAAAAAAAAAAAAAAAAAAAAAAAAAAAAAAAAAAAAAAAAAAAA"
+			"AAAAAAAAAAAAAAAAAAAAAAAAAAAAAAAAAAAAAAAAAAAAAAAAAAAAAAAAAAAAAAAAAAAAAAAAAAAA"
+			"AAAAAAAAAAAAAAAAAAAAAAAAAAAAAAAAAAAAAAAAAAAAAAAAAAAAAAAAAAAAAAAAAAAAAAAAAAAA"
+			"AAAAAAAAAAAAAAAAAAAAAAAAAAAAAAAAAAAAAAAAAAAAAAAAAAAAAAAAAAAAAAAAAAAAAAAAAAAA"
+			"AAAAAAAAAAAAAAAAAAAAAAAAAAAAAAAAAAAAAAAAAAAAAAAAAAAAAAAAAAAAAAAAAAAAAAAAAAAA"
+			"AAAAAAAAAAAAAAAAAAAAAAAAAAAAAAAAAAAAAAAAAAAAAAAAAAAAAAAAAAAAAAAAAAAAAAAAAAAA"
+			"AAAAAAAAAAAAAAAAAAAAAAAAAAAAAAAAAAAAAAAAAAAAAAAAAAAAAAAAAAAAAAAAAAAAAAAAAAAA"
+			"AAAAAAAAAAAAAAAAAAAAAAAAAAAAAAAAAAAAAAAAAAAAAAAAAAAAAAAAAAAAAAAAAAAAAAAAAAAA"
+			"AAAAAAAAAAAAAAAAAAAAAAAAAAAAAAAAAAAAAAAAAAAAAAAAAAAAAAAAAAAAAAAAAAAAAAAAAAAA"
+			"AAAAAAAAAAAAAAAAAAAAAAAAAAAAAAAAAAAAAAAAAAAAAAAAAAAAAAAAAAAAAAAAAAAAAAAAAAAA"
+			"AAAAAAAAAAAAAAAAAAAAAAAAAAAAAAAAAAAAAAAAAAAAAAAAAAAAAA=="
 		)
 	)
@@
 			"AAAAAAAAAAAwAAAAMAAAANB8AAAAAAAAcAAAAAAAAABhoiIBGlYAAAAAAAAAAAAAAAAAAAAAAAAA"
 			"AAAABAAAAAgAAAAwAAAAMAAAAMAAAAABAAAAAAAAAAAAAAAAAAAAUDyxh8p/AAAAAAAAAAAAAAAA"
-			"AAAAAAAAAQAAAAAAAABAfQAAAAAAAA=="
+			"AAAAAAAAAQAAAAAAAABAfQAAAAAAAAAAAAAAAAAAAAAAAAAAAAAAAAAAAAAAAAAAAAAAAAAAAAAA"
+			"AAAAAAAAAAAAAAAAAAAAAAAAAAAAAAAAAAAAAAAAAAAAAAAAAAAAAAAAAAAAAAAAAAAAAAAAAAAA"
+			"AAAAAAAAAAAAAAAAAAAAAAAAAAAAAAAAAAAAAAAAAAAAAAAAAAAAAAAAAAAAAAAAAAAAAAAAAAAA"
+			"AAAAAAAAAAAAAAAAAAAAAAAAAAAAAAAAAAAAAAAAAAAAAAAAAAAAAAAAAAAAAAAAAAAAAAAAAAAA"
+			"AAAAAAAAAAAAAAAAAAAAAAAAAAAAAAAAAAAAAAAAAAAAAAAAAAAAAAAAAAAAAAAAAAAAAAAAAAAA"
+			"AAAAAAAAAAAAAAAAAAAAAAAAAAAAAAAAAAAAAAAAAAAAAAAAAAAAAAAAAAAAAAAAAAAAAAAAAAAA"
+			"AAAAAAAAAAAAAAAAAAAAAAAAAAAAAAAAAAAAAAAAAAAAAAAAAAAAAAAAAAAAAAAAAAAAAAAAAAAA"
+			"AAAAAAAAAAAAAAAAAAAAAAAAAAAAAAAAAAAAAAAAAAAAAAAAAAAAAAAAAAAAAAAAAAAAAAAAAAAA"
+			"AAAAAAAAAAAAAAAAAAAAAAAAAAAAAAAAAAAAAAAAAAAAAAAAAAAAAAAAAAAAAAAAAAAAAAAAAAAA"
+			"AAAAAAAAAAAAAAAAAAAAAAAAAAAAAAAAAAAAAAAAAAAAAAAAAAAAAAAAAAAAAAAAAAAAAAAAAAAA"
+			"AAAAAAAAAAAAAAAAAAAAAAAAAAAAAAAAAAAAAAAAAAAAAAAAAAAAAAAAAAAAAAAAAAAAAAAAAAAA"
+			"AAAAAAAAAAAAAAAAAAAAAAAAAAAAAAAAAAAAAAAAAAAAAAAAAAAAAAAAAAAAAAAAAAAAAAAAAAAA"
+			"AAAAAAAAAAAAAAAAAAAAAAAAAAAAAAAAAAAAAAAAAAAAAAAAAAAAAAAAAAAAAAAAAAAAAAAAAAAA"
+			"AAAAAAAAAAAAAAAAAAAAAAAAAAAAAAAAAAAAAAAAAAAAAAAAAAAAAAAAAAAAAAAAAAAAAAAAAAAA"
+			"AAAAAAAAAAAAAAAAAAAAAAAAAAAAAAAAAAAAAAAAAAAAAAAAAAAAAAAAAAAAAAAAAAAAAAAAAAAA"
+			"AAAAAAAAAAAAAAAAAAAAAAAAAAAAAAAAAAAAAAAAAAAAAAAAAAAAAAAAAAAAAAAAAAAAAAAAAAAA"
+			"AAAAAAAAAAAAAAAAAAAAAAAAAAAAAAAAAAAAAAAAAAAAAAAAAAAAAAAAAAAAAAAAAAAAAAAAAAAA"
+			"AAAAAAAAAAAAAAAAAAAAAAAAAAAAAAAAAAAAAAAAAAAAAAAAAAAAAAAAAAAAAAAAAAAAAAAAAAAA"
+			"AAAAAAAAAAAAAAAAAAAAAAAAAAAAAA=="
 		)
 	)
@@
 			"AAAAAAAAAAAAAAAAAAAAAAAAAAAAAAAAAAAAAAEAAAAAAAAAAAAAAAAAAAAAAAAAAAAAAAAAAAAA"
 			"AAAAAAAAAAAAAAAAAAAAAAAAAAAAAAAAAAAAAAAAAAAAAAAAAAAAAAAAAGTO///Sl///AAAAAL6h"
-			"//8AAAAAAAAAAAAAAAAAAAAAAAAAAAAAAAAAAAAAAAAAAAAAAAAAAAAAAAAAAAAAAAAAAAAAAA=="
+			"//8AAAAAAAAAAAAAAAAAAAAAAAAAAAAAAAAAAAAAAAAAAAAAAAAAAAAAAAAAAAAAAAAAAAAAAAAA"
+			"AAAAAAAAAAAAAAAAAAAAAAAAAAAAAAAAAAAAAAAAAAAAAAAAAAAAAAAAAAAAAAAAAAAAAAAAAAAA"
+			"AAAAAAAAAAAAAAAAAAAAAAAAAAAAAAAAAAAAAAAAAAAAAAAAAAAAAAAAAAAAAAAAAAAAAAAAAAAA"
+			"AAAAAAAAAAAAAAAAAAAAAAAAAAAAAAAAAAAAAAAAAAAAAAAAAAAAAAAAAAAAAAAAAAAAAAAAAAAA"
+			"AAAAAAAAAAAAAAAAAAAAAAAAAAAAAAAAAAAAAAAAAAAAAAAAAAAAAAAAAAAAAAAAAAAAAAAAAAAA"
+			"AAAAAAAAAAAAAAAAAAAAAAAAAAAAAAAAAAAAAAAAAAAAAAAAAAAAAAAAAAAAAAAAAAAAAAAAAAAA"
+			"AAAAAAAAAAAAAAAAAAAAAAAAAAAAAAAAAAAAAAAAAAAAAAAAAAAAAAAAAAAAAAAAAAAAAAAAAAAA"
+			"AAAAAAAAAAAAAAAAAAAAAAAAAAAAAAAAAAAAAAAAAAAAAAAAAAAAAAAAAAAAAAAAAAAAAAAAAAAA"
+			"AAAAAAAAAAAAAAAAAAAAAAAAAAAAAAAAAAAAAAAAAAAAAAAAAAAAAAAAAAAAAAAAAAAAAAAAAAAA"
+			"AAAAAAAAAAAAAAAAAAAAAAAAAAAAAAAAAAAAAAAAAAAAAAAAAAAAAAAAAAAAAAAAAAAAAAAAAAAA"
+			"AAAAAAAAAAAAAAAAAAAAAAAAAAAAAAAAAAAAAAAAAAAAAAAAAAAAAAAAAAAAAAAAAAAAAAAAAAAA"
+			"AAAAAAAAAAAAAAAAAAAAAAAAAAAAAAAAAAAAAAAAAAAAAAAAAAAAAAAAAAAAAAAAAAAAAAAAAAAA"
+			"AAAAAAAAAAAAAAAAAAAAAAAAAAAAAAAAAAAAAAAAAAAAAAAAAAAAAAAAAAAAAAAAAAAAAAAAAAAA"
+			"AAAAAAAAAAAAAAAAAAAAAAAAAAAAAAAAAAAAAAAAAAAAAAAAAAAAAAAAAAAAAAAAAAAAAAAAAAAA"
+			"AAAAAAAAAAAAAAAAAAAAAAAAAAAAAAAAAAAAAAAAAAAAAAAAAAAAAAAAAAAAAAAAAAAAAAAAAAAA"
+			"AAAAAAAAAAAAAAAAAAAAAAAAAAAAAAAAAAAAAAAAAAAAAAAAAAAAAAAAAAAAAAAAAAAAAAAAAAAA"
+			"AAAAAAAAAAAAAAAAAAAAAAAAAAAAAAAAAAAAAAAAAAAAAAAAAAAAAAAAAAAAAAAAAAAAAAAAAAAA"
+			"AAAAAAAAAAAAAAAAAAAAAAAAAAAAAAAAAAAAAAAAAAAAAAAAAAAAAAAAAAAAAAAAAAAAAAAAAAAA"
+			"AAAAAAAAAAAAAAAAAAAAAAAAAAAAAAAAAAAAAAAAAAAAAAAAAAAAAAAAAAAAAAAAAAAAAAAAAA=="
 		)
 	)
@@
 			"AGIAAABhAAAAdAAAAHQAAABlAAAAcgAAAHkAAABwAAAAYQAAAGMAAABrAAAALwAAAG4AAAByAAAA"
 			"ZQAAAGYAAAAtAAAAYgAAAGEAAAB0AAAAdAAAAGUAAAByAAAAeQAAAGYAAAByAAAAbwAAAG4AAAB0"
-			"AAAALQAAAGQAAAAxAAAALwAAAG4AAA=="
+			"AAAALQAAAGQAAAAxAAAALwAAAG4AAGk5KzE3L25VQUFJRGxWSzlSL1hSY1hHNXVya2xSQ0hIcXIr"
+			"dGRBZGcyS3dvek1uOS8velp0MjR3YU0zcngwaVZ5OGNLRkMwSUk3OUtsNVVwQ2ZQeXoxOG5YWkdN"
+			"K1BxVnIxNmxkdTA3dGhvMGF2dm5XV3lQQ1F2OWVKeUhoK2RjQkFBQ1cwNjc5SzNmdjNvMDlmTmk0"
+			"MkxSWk0xZFgxNTNmZmFkVVZ3Q0traldHR1ZsQTJiTHlPRDA5WFFoUnNtUkoxNy91NHh3VEhmUHMr"
+			"empuYS9JenRIejU3NHNJYjk2NFdiQkZBQUNBZWJWL3BiMi92LytIOCtmbjVPVElSU2NucDU2OWVr"
+			"WkdSQ2JFOC9OSHdQWlpSWmpadDNldlhxL1BXOSs5YTVjOHJsQytnaEJDbzlHRXZQcXFWSG40OE9G"
+			"SFQ3cnhZa3BLU25wYWVuNG5QN085djdlV2xUWEtWd0FBUUVGT1RrN1RaODVJaUU4dytTcytOR3hr"
+			"cVZLbHdrSkhQSGp3UUtuZUFCUU5xN2cxODhqUU1EZDN0NDRkT3pWdTByaDgrUXJGU3hUL0l6VTFl"
+			"bC8wRjVzMnlYUHExcThuRFhyMzZiMWw4Mlpwdkg3ZHV2VDA5T0RPd1pVclYwNU4vZVAzMzMrTGlZ"
+			"NDUvc3N2MnlJaUdqWnFtTi9Kc2w5UC83cG93VUloeE1OSEQ4K2ZPMjk4bTJacEp5NEFBTEFHSFR0"
+			"MTZ2L3ZmNjlaSFY2MWF0VWVQWHRLeFJJZUpUNWRzcmovTy8xR0RCdTJlczBhQndlcitHNEhnQ1Zv"
+			"REFhRDBqMklPalZyUGZ1dUk2OTA2TEFxZkxYOHNsZVBuc2QvK2VVWjg0M3p5Zk5Qcmw0MTBQZzhk"
+			"VjVWcWxiNS9zY2ZqVytTOW84eTB0TTNmN001SXlQaitUOENBS3BnTUJoaVltTE9KaVEwYk5USTN0"
+			"NWU2WFpza0l1emM2M2F0WjJjbkJUczRjNmRPeGN2WGpTNXd0NXlIQjBkYTlXcVZheFlzWHg5S2pj"
+			"MzkvdW9xSlNVbEdVclZnUjNEcGJyV3pkdm1UaGhRclZxMVRwMjZtVHlETzVDdW5ualJuSnljdEY4"
+			"LytUdTVsYXJkbTA3TzZ2WVNnUGI1dVRrOU5xL1hpOVhycHpTamVTUENzSk1ZR0RncWpYaDhpM0Zo"
+			"QkNabVpsREJnNktqWTE5MmtlTXc4enpUMzUybVBFUENGaTJmRm45QmcyZS9iV1lHRGRtYk1UMjdm"
+			"bjZDQUFBeUMrTlJtTm5aN2Q2elpvMmJkdkl4YzgvKyt6akR6OVNzQ3RBWGFwWHIvN0Q3bDMvUE0r"
+			"YVdFWFFuelpqK2t2Tlg4cjd3eWN2TA=="
 		)
 	)
