File: nref-ports-two/nref-ports-two.kicad_sch (KiCad schematic)
At the start: 117 parts, among them J1 USB_C_Receptacle, J2 USB_C_Receptacle, J3 USB3_A, J4 HD0919MSMTTR, J5 Conn_01x20, J6 Conn_01x12_Pin, J7 Conn_01x04, U1 TUSB8041, U10 TPD4E02B04DQA, U11 TPD12S521, U12 LM2830XQMFE/NOPB, U13 LM2830XQMFE/NOPB, U2 HD3SS3220IRNHT, U3 TPD4E02B04DQA, U4 TPD4E02B04DQA, U5 TPD4E02B04DQA, U6 TPD4E02B04DQA, U7 TPD4E02B04DQA, U8 TPD4E02B04DQA, U9 TPD4E02B04DQA, Y1 24MHz

Commit message: add various notes in schematics
Other:
- note added: "TODO: experimentally fitted 10k to boost to 1.2V"
Changed lines of the file:
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@@
+		)
+	)
+	(text "TODO: experimentally fitted 10k\nto boost to 1.2V"
+		(exclude_from_sim no)
+		(at 304.8 163.83 0)
+		(effects
+			(font
+				(size 1.27 1.27)
+			)
 		)
 	)
