File: nref-ports-two/nref-ports-two.kicad_sch (KiCad schematic)
At the start: 109 parts, among them J1 USB_C_Receptacle, J2 USB_C_Receptacle, J3 USB3_A, J4 HD0919MSMTTR, J5 Conn_01x20, J6 Conn_01x12_Pin, U1 TUSB8041, U10 TPD4E02B04DQA, U11 TPD12S521, U12 LM2830XQMFE/NOPB, U13 LM2830XQMFE/NOPB, U2 HD3SS3220IRNHT, U3 TPD4E02B04DQA, U4 TPD4E02B04DQA, U5 TPD4E02B04DQA, U6 TPD4E02B04DQA, U7 TPD4E02B04DQA, U8 TPD4E02B04DQA, U9 TPD4E02B04DQA, Y1 24MHz

Commit message: ports-two: hdmi routing snapshot
Parts:
- removed R19, R20: 0, Resistor_SMD:R_0402_1005Metric, symbol Device:R_Small
- added H1, H2: MountingHole_Pad, MountingHole:MountingHole_2.2mm_M2_Pad, symbol Mechanical:MountingHole_Pad
- added R39, R40, R43, R44: 22k, Resistor_SMD:R_0402_1005Metric, symbol Device:R_Small
- added TP1, TP2: TestPoint, TestPoint:TestPoint_Pad_1.0x1.0mm, symbol Connector:TestPoint
- C1, C2, C33, C34, C35, C36, C37, C38: footprint Capacitor_SMD:C_0603_1608Metric -> Capacitor_SMD:C_0402_1005Metric
- R26, R27, R28, R29, R30, R31, R32, R33, R34: footprint Resistor_SMD:R_0603_1608Metric -> Resistor_SMD:R_0402_1005Metric
Connections:
- net +5V: now also R39.1, R40.1, R43.1, R44.1
- net CC1: now also R43.2
- net CC2: now also R44.2
- net GND: now also H1.1, H2.1
- net at U2.25 (SDA/OUT1): now also TP2.1
- net at U2.26 (SCL/OUT2): now also TP1.1
- net at J2.A5 (CC1), U6.1 (IO1), U6.10 (IO1): now also R39.2
- net at J2.B5 (CC2), U6.2 (IO2), U6.9 (IO2): now also R40.2
- no-connect marks 22 -> 20
Other:
- note removed: "TODO: CC resistors?"
- note removed: "TODO: test points?"

Commit message: ports two: usb snapshot
Connections:
- net USB2A_DN is gone; now on net USB2_DN: J6.1 (Pin_1)
- net USB2A_DP is gone; now on net USB2_DP: J6.2 (Pin_2)
- net USBH_1A_RXN: now also U9.5 (IO4), U9.6 (IO4); no longer U9.4 (IO3), U9.7 (IO3)
- net USBH_1A_RXP: now also U9.4 (IO3), U9.7 (IO3); no longer U9.5 (IO4), U9.6 (IO4)
- net USBH_1B_RXN: now also U1.29 (USB_SSRXP_DN4); no longer U1.22 (USB_SSRXP_DN3)
- net USBH_1B_RXP: now also U1.30 (USB_SSRXM_DN4); no longer U1.23 (USB_SSRXM_DN3)
- net USBH_1B_TXN: now also U1.27 (USB_SSTXM_DN4); no longer U1.19 (USB_SSTXP_DN3)
- net USBH_1B_TXP: now also U1.26 (USB_SSTXP_DN4); no longer U1.20 (USB_SSTXM_DN3)
- net USBH_2B_AC_TXN: now also U5.5 (IO4), U5.6 (IO4); no longer U5.4 (IO3), U5.7 (IO3)
- net USBH_2B_AC_TXP: now also U5.4 (IO3), U5.7 (IO3); no longer U5.5 (IO4), U5.6 (IO4)
- net USBH_2B_RXN: now also U1.22 (USB_SSRXP_DN3); no longer U1.29 (USB_SSRXP_DN4)
- net USBH_2B_RXP: now also U1.23 (USB_SSRXM_DN3); no longer U1.30 (USB_SSRXM_DN4)
- net USBH_2B_TXN: now also U1.20 (USB_SSTXM_DN3); no longer U1.26 (USB_SSTXP_DN4)
- net USBH_2B_TXP: now also U1.19 (USB_SSTXP_DN3); no longer U1.27 (USB_SSTXM_DN4)
Other:
- note added: "TODO: missing RC!"
- note added: "TODO: unused"
- note removed: "N/P swapped"
- note removed: "to kbd/trackball"
- note removed: "to modem"

Commit message: port board two fully routed
Parts:
- removed R10: 0, Resistor_SMD:R_0402_1005Metric, symbol Device:R_Small
- added C43: 10uF, Capacitor_SMD:C_0603_1608Metric, symbol Device:C_Small
- C12, C16: footprint Capacitor_SMD:C_0402_1005Metric -> Capacitor_SMD:C_0603_1608Metric
- R3: value 100k -> 1M; LCSC C60491 -> (none); Manufacturer_No RC0402FR-07100KL -> RC0402FR-071ML
Connections:
- net CC1: no longer R15.1
- net CC2: no longer R14.1
- net GND: now also C43.2; no longer R3.2
- net USBH_3V3: now also R3.2
- net ~{USBH_RESET}: now also U1.50 (GRSTz), C43.1
- net MUXCC2: now reaches J2.B5 (CC2), R40.2, U6.2 (IO2), U6.9 (IO2)
- net MUXCC2: now also R14.1
- net MUXCC1: now reaches J2.A5 (CC1), R39.2, U6.1 (IO1), U6.10 (IO1)
- net MUXCC1: now also R15.1
Other:
- note added: "Hub RC reset circuit"
- note added: "TODO: unused, break out for camera"
- note removed: "TODO: missing RC!"
- note removed: "TODO: unused"

Commit message: ports two bom adjustments
Parts:
- added H3: BADGE, footprints:nref-ports-two-badge, symbol Mechanical:MountingHole
- added J7: Conn_01x04, Connector_JST:JST_SH_SM04B-SRSS-TB_1x04-1MP_P1.00mm_Horizontal, symbol Connector_Generic:Conn_01x04
- C1, C2: LCSC C107040 -> (none)
- C10, C11, C13, C14, C15, C18, C21, C22, C23, C24, C27, C28, C29, C3, C30, C4, C5, C6, C7, C8, C9: LCSC C1525 -> (none)
- C12, C16: LCSC C315248 -> (none); Manufacturer_No CL05A106MP5NUNC -> CL10A106MO8NQNC
- C17, C19, C20, C25, C26, C31, C32, C40, C42: Manufacturer (none) -> TDK; Manufacturer_No (none) -> C3216X5R1E476M160AC
- C33, C34, C35, C36, C37, C38: Checked y -> (none); Distributor Mouser -> (none); Manufacturer Yageo -> Samsung; Manufacturer_No CC0603JPX7R9BB104 -> CL05B104KO5NNNC
- C39, C41: LCSC C86295 -> (none)
- C43: LCSC C92487 -> (none)
- D1, J3, U11: Checked y -> (none); Distributor Mouser -> (none)
- D2, D3: LCSC C426863 -> (none)
- FB1, FB2: LCSC C88980 -> (none)
- H1, H2, TP1, TP2: Manufacturer (none) -> DNP; Manufacturer_No (none) -> DNP; now not fitted
- J1, J2: LCSC C134092 -> (none)
- J4: Manufacturer (none) -> CUI; Manufacturer_No HD0919MSMTTR -> HD09-19-MSMT-TR
- L1, L2: LCSC C337905 -> (none); Manufacturer_No LQH32PN3R3NN0L -> DFE32CAH3R3MR0L
- R1: LCSC C844710 -> (none); Manufacturer Vishay -> Vishay Dale
- R11: LCSC C242160 -> (none); Manufacturer Panasonic -> Yageo; Manufacturer_No ERJ2GE0R00X -> RC0402FR-7D10KL
- R12: value 900k -> 909k; LCSC C242160 -> (none); Manufacturer Panasonic -> Bourns; Manufacturer_No ERJ2GE0R00X -> CR0402-FX-9093GLF
- R13, R18, R22, R23, R24: LCSC C242160 -> (none); Manufacturer Panasonic -> Bourns; Manufacturer_No ERJ2GE0R00X -> CR0402-JW-204GLF
- R14, R15, R16, R17, R21, R25: LCSC C242160 -> (none); Manufacturer Panasonic -> Vishay Dale; Manufacturer_No ERJ2GE0R00X -> CRCW04020000Z0EDC
- R2: LCSC C144787 -> (none); Manufacturer_No AC0402FR-071ML -> RC0402FR-071ML
- R26, R30: Checked y -> (none); Distributor Mouser -> (none); Manufacturer_No RC0603FR-0710KL -> RC0402FR-7D10KL
- R27, R29: Checked y -> (none); Distributor Mouser -> (none); Manufacturer_No RC0603FR-074K7L -> RC0402FR-074K7L
- R28: Checked y -> (none); Distributor Mouser -> (none); Manufacturer Bourns -> Vishay Dale; Manufacturer_No CR0603-FX-2702ELF -> CRCW040227K0FKEDHP
- R31: Checked y -> (none); Distributor Mouser -> (none); Manufacturer Vishay Dale -> Yageo; Manufacturer_No CRCW0603100KJNEAC -> RC0402FR-07100KL
- R32, R33, R34: Checked y -> (none); Distributor Mouser -> (none); Manufacturer Vishay Dale -> Panasonic; Manufacturer_No CRCW060347K0FKEAC -> ERA-2AEB473X
- R35, R36: LCSC C242160 -> (none); Manufacturer Panasonic -> Yageo; Manufacturer_No ERJ2GE0R00X -> RC0402FR-07100KL
- R37: LCSC C95598 -> (none); Manufacturer UNI-ROYAL -> Yageo; Manufacturer_No 0402WGF8251TCE -> NT0402BRD078K25L
- R38, R42, R6: LCSC C60490 -> (none); Manufacturer_No RC0402FR-0710KL -> RC0402FR-7D10KL
- R39, R40, R43, R44: Manufacturer (none) -> Panasonic; Manufacturer_No (none) -> ERA-2AED223X
- R4: LCSC C26989 -> (none); Manufacturer UNI-ROYAL -> Bourns; Manufacturer_No 0402WGF9092TCE -> CR0402-FX-9092GLF
- R41: LCSC C95598 -> (none); Manufacturer UNI-ROYAL -> Vishay Dale; Manufacturer_No 0402WGF8251TCE -> TNPW040245K3FHED
- R5, R8, R9: LCSC C105871 -> (none)
- R7: LCSC C321660 -> (none); Manufacturer FH -> Bourns; Manufacturer_No RC-02W9531FT -> CR0402-FX-9531GLF
- U10, U3, U4, U5, U6, U7, U8, U9: LCSC C2841426 -> (none)
- U12, U13: LCSC C2072452 -> (none)
- U2: AVAILABILITY Good -> (none); Availability In Stock -> (none); Check_prices https://www.snapeda.com/parts/HD3SS3220IRNHT/Texas+Instrume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 -> (none); DESCRIPTION Super Speed Type-C DRP Port Controller USB 3.1 3.3V/5V T/R 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 -> (none); Description_1 10-Gbps USB 3.1 Type-C 2:1 mux with DRP Controller -> (none); MF Texas Instruments -> (none); MP HD3SS3220IRNHT -> (none); Manufacturer (none) -> Texas Instruments; Manufacturer_No (none) -> HD3SS3220IRNHT; PACKAGE WQFN-30 Texas Instruments -> (none); PART_REV C -> (none); PRICE 3.26 USD -> (none); Package WQFN-30 Texas Instruments -> (none); Price None -> (none); Purchase-URL https://www.snapeda.com/api/url_track_click_mouser/?unipart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 -> (none); STANDARD IPC-7351B -> (none); SnapEDA_Link https://www.snapeda.com/parts/HD3SS3220IRNHT/Texas+Instrume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 -> (none)
- Y1: LCSC C91744 -> (none)
Connections:
- net +5V: now also J7.4 (Pin_4)
- net GND: now also J7.1 (Pin_1)
- net USBH_4_DN: now also J7.3 (Pin_3)
- net USBH_4_DP: now also J7.2 (Pin_2)
Other:
- note removed: "TODO: unused, break out for camera"

Commit message: add latest PCB updates
Other:
- note added: "TODO: DNP @ 22k"
- note added: "TODO: flipped!"
- moved on the sheet: J5, J6, J7, R1

Commit message: snapshot before merge
Other:
- note added: "TODO/FIXME: sda/scl flipped vs rcore+hdmiedp!"
Changed lines of the file:
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@@
 (kicad_sch
-	(version 20231120)
+	(version 20250114)
 	(generator "eeschema")
-	(generator_version "8.0")
+	(generator_version "9.0")
 	(paper "A2")
+	(text "TODO: are these pullups required here or are they already on the mb?"
+		(exclude_from_sim no)
+		(at 261.62 144.78 0)
+		(effects
+			(font
+				(size 1.27 1.27)
+			)
+		)
+	)
+	(text "USB3 to port farm 2\n(flipped)"
+		(exclude_from_sim no)
+		(at 267.97 -92.71 0)
+		(effects
+			(font
+				(size 1.27 1.27)
+			)
+			(justify left bottom)
+		)
+	)
+	(text "Hub RC reset circuit"
+		(exclude_from_sim no)
+		(at 382.905 200.66 0)
+		(effects
+			(font
+				(size 1.27 1.27)
+			)
+		)
+	)
+	(text "=1.095V"
+		(exclude_from_sim no)
+		(at 302.26 173.99 0)
+		(effects
+			(font
+				(size 1.27 1.27)
+			)
+			(justify left bottom)
+		)
+	)
+	(text "=3.3V"
+		(exclude_from_sim no)
+		(at 302.26 226.06 0)
+		(effects
+			(font
+				(size 1.27 1.27)
+			)
+			(justify left bottom)
+		)
+	)
+	(text "TODO: double check ENN_CC, PORT"
+		(exclude_from_sim no)
+		(at 53.34 208.28 0)
+		(effects
+			(font
+				(size 1.27 1.27)
+			)
+		)
+	)
+	(text "USB-C port 1"
+		(exclude_from_sim no)
+		(at 59.69 289.56 0)
+		(effects
+			(font
+				(size 2.54 2.54)
+			)
+			(justify left bottom)
+		)
+	)
+	(text "HDMI to port farm\n(flipped)"
+		(exclude_from_sim no)
+		(at 218.186 -92.71 0)
+		(effects
+			(font
+				(size 1.27 1.27)
+			)
+			(justify left bottom)
+		)
+	)
+	(text "TODO: DNP @ 22k"
+		(exclude_from_sim no)
+		(at 303.784 290.322 0)
+		(effects
+			(font
+				(size 1.27 1.27)
+			)
+		)
+	)
+	(text "1A"
+		(exclude_from_sim no)
+		(at 270.51 165.1 0)
+		(effects
+			(font
+				(size 1.27 1.27)
+			)
+			(justify left bottom)
+		)
+	)
+	(text "TODO: fuses / current limit"
+		(exclude_from_sim no)
+		(at 278.13 269.24 0)
+		(effects
+			(font
+				(size 1.27 1.27)
+			)
+		)
+	)
+	(text "TODO/FIXME: sda/scl flipped vs rcore+hdmiedp!"
+		(exclude_from_sim no)
+		(at 197.866 -87.884 0)
+		(effects
+			(font
+				(size 1.27 1.27)
+			)
+		)
+	)
+	(text "TODO: fuses / current limit"
+		(exclude_from_sim no)
+		(at 140.97 320.675 0)
+		(effects
+			(font
+				(size 1.27 1.27)
+			)
+		)
+	)
+	(text "1A"
+		(exclude_from_sim no)
+		(at 270.51 217.17 0)
+		(effects
+			(font
+				(size 1.27 1.27)
+			)
+			(justify left bottom)
+		)
+	)
+	(text "USB-C port 2"
+		(exclude_from_sim no)
+		(at 256.54 289.56 0)
+		(effects
+			(font
+				(size 2.54 2.54)
+			)
+			(justify left bottom)
+		)
+	)
+	(text "Port\nProtection"
+		(exclude_from_sim no)
+		(at 138.43 85.09 0)
+		(effects
+			(font
+				(size 1.27 1.27)
+			)
+			(justify left bottom)
+		)
+	)
+	(text "USB Hub"
+		(exclude_from_sim no)
+		(at 471.17 35.56 0)
+		(effects
+			(font
+				(size 2.54 2.54)
+			)
+			(justify left bottom)
+		)
+	)
+	(text "TODO: flipped!"
+		(exclude_from_sim no)
+		(at 193.04 302.006 0)
+		(effects
+			(font
+				(size 1.27 1.27)
+			)
+		)
+	)
+	(text "https://www.ti.com/lit/ds/symlink/hd3ss3220.pdf?ts=1718344395887"
+		(exclude_from_sim no)
+		(at 102.87 182.88 0)
+		(effects
+			(font
+				(size 1.27 1.27)
+			)
+		)
+	)
 	(junction
 		(at 172.72 97.79)
@@
 		)
 	)
-	(text "TODO: are these pullups required here or are they already on the mb?"
-		(exclude_from_sim no)
-		(at 261.62 144.78 0)
-		(effects
-			(font
-				(size 1.27 1.27)
-			)
-		)
-	)
-	(text "USB3 to port farm 2\n(flipped)"
-		(exclude_from_sim no)
-		(at 267.97 -92.71 0)
-		(effects
-			(font
-				(size 1.27 1.27)
-			)
-			(justify left bottom)
-		)
-	)
-	(text "Hub RC reset circuit"
-		(exclude_from_sim no)
-		(at 382.905 200.66 0)
-		(effects
-			(font
-				(size 1.27 1.27)
-			)
-		)
-	)
-	(text "=1.095V"
-		(exclude_from_sim no)
-		(at 302.26 173.99 0)
-		(effects
-			(font
-				(size 1.27 1.27)
-			)
-			(justify left bottom)
-		)
-	)
-	(text "=3.3V"
-		(exclude_from_sim no)
-		(at 302.26 226.06 0)
-		(effects
-			(font
-				(size 1.27 1.27)
-			)
-			(justify left bottom)
-		)
-	)
-	(text "TODO: double check ENN_CC, PORT"
-		(exclude_from_sim no)
-		(at 53.34 208.28 0)
-		(effects
-			(font
-				(size 1.27 1.27)
-			)
-		)
-	)
-	(text "USB-C port 1"
-		(exclude_from_sim no)
-		(at 59.69 289.56 0)
-		(effects
-			(font
-				(size 2.54 2.54)
-			)
-			(justify left bottom)
-		)
-	)
-	(text "HDMI to port farm\n(flipped)"
-		(exclude_from_sim no)
-		(at 218.186 -92.71 0)
-		(effects
-			(font
-				(size 1.27 1.27)
-			)
-			(justify left bottom)
-		)
-	)
-	(text "TODO: DNP @ 22k"
-		(exclude_from_sim no)
-		(at 303.784 290.322 0)
-		(effects
-			(font
-				(size 1.27 1.27)
-			)
-		)
-	)
-	(text "1A"
-		(exclude_from_sim no)
-		(at 270.51 165.1 0)
-		(effects
-			(font
-				(size 1.27 1.27)
-			)
-			(justify left bottom)
-		)
-	)
-	(text "TODO: fuses / current limit"
-		(exclude_from_sim no)
-		(at 278.13 269.24 0)
-		(effects
-			(font
-				(size 1.27 1.27)
-			)
-		)
-	)
-	(text "TODO: fuses / current limit"
-		(exclude_from_sim no)
-		(at 140.97 320.675 0)
-		(effects
-			(font
-				(size 1.27 1.27)
-			)
-		)
-	)
-	(text "1A"
-		(exclude_from_sim no)
-		(at 270.51 217.17 0)
-		(effects
-			(font
-				(size 1.27 1.27)
-			)
-			(justify left bottom)
-		)
-	)
-	(text "USB-C port 2"
-		(exclude_from_sim no)
-		(at 256.54 289.56 0)
-		(effects
-			(font
-				(size 2.54 2.54)
-			)
-			(justify left bottom)
-		)
-	)
-	(text "Port\nProtection"
-		(exclude_from_sim no)
-		(at 138.43 85.09 0)
-		(effects
-			(font
-				(size 1.27 1.27)
-			)
-			(justify left bottom)
-		)
-	)
-	(text "USB Hub"
-		(exclude_from_sim no)
-		(at 471.17 35.56 0)
-		(effects
-			(font
-				(size 2.54 2.54)
-			)
-			(justify left bottom)
-		)
-	)
-	(text "TODO: flipped!"
-		(exclude_from_sim no)
-		(at 193.04 302.006 0)
-		(effects
-			(font
-				(size 1.27 1.27)
-			)
-		)
-	)
-	(text "https://www.ti.com/lit/ds/symlink/hd3ss3220.pdf?ts=1718344395887"
-		(exclude_from_sim no)
-		(at 102.87 182.88 0)
-		(effects
-			(font
-				(size 1.27 1.27)
-			)
-		)
-	)
 	(label "USBH_1A_AC_TXN"
 		(at 334.01 341.63 0)
-		(fields_autoplaced yes)
 		(effects
 			(font
@@
 	(label "USB3_1_SSTXCP"
 		(at 487.68 316.23 0)
-		(fields_autoplaced yes)
 		(effects
 			(font
@@
 	(label "USBH_1B_AC_TXP"
 		(at 334.01 359.41 0)
-		(fields_autoplaced yes)
 		(effects
 			(font
@@
 	(label "USBH_2A_AC_TXN"
 		(at 137.16 341.63 0)
-		(fields_autoplaced yes)
 		(effects
 			(font
@@
 	(label "USBH_2B_AC_TXP"
 		(at 137.16 359.41 0)
-		(fields_autoplaced yes)
 		(effects
 			(font
@@
 	(label "USBH_2B_AC_TXN"
 		(at 137.16 356.87 0)
-		(fields_autoplaced yes)
 		(effects
 			(font
@@
 	(label "USBH_2A_AC_TXP"
 		(at 137.16 344.17 0)
-		(fields_autoplaced yes)
 		(effects
 			(font
@@
 	(label "USB3_1_SSTXCN"
 		(at 487.68 313.69 0)
-		(fields_autoplaced yes)
 		(effects
 			(font
@@
 	(label "USBH_1B_AC_TXN"
 		(at 334.01 356.87 0)
-		(fields_autoplaced yes)
 		(effects
 			(font
@@
 	(label "USBH_1A_AC_TXP"
 		(at 334.01 344.17 0)
-		(fields_autoplaced yes)
 		(effects
 			(font
@@
 		)
 	)
+	(embedded_fonts no)
 )

Commit message: add current notes on various schematics
Other:
- note added: "TODO: change to 10k!"
- note added: "TODO: missing caps on TX"
- note added: "TODO: six layer design, power close to diff pairs is questionable"
- note added: "TODO: works only in one orientation"
- note added: "USB3 to port farm 2"
- note removed: "TODO: are these pullups required here or are they already on the mb?"
- note removed: "USB3 to port farm 2 (flipped)"
Changed lines of the file:
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@@
 	(generator_version "9.0")
 	(paper "A2")
-	(text "TODO: are these pullups required here or are they already on the mb?"
-		(exclude_from_sim no)
-		(at 261.62 144.78 0)
-		(effects
-			(font
-				(size 1.27 1.27)
-			)
-		)
-	)
-	(text "USB3 to port farm 2\n(flipped)"
+	(text "USB3 to port farm 2"
 		(exclude_from_sim no)
 		(at 267.97 -92.71 0)
@@
 			)
 			(justify left bottom)
+		)
+	)
+	(text "TODO: change to 10k!"
+		(exclude_from_sim no)
+		(at 267.97 105.41 0)
+		(effects
+			(font
+				(size 1.27 1.27)
+			)
 		)
 	)
@@
 		)
 	)
+	(text "TODO: six layer design, power close to diff pairs is questionable"
+		(exclude_from_sim no)
+		(at 419.1 132.08 0)
+		(effects
+			(font
+				(size 1.27 1.27)
+			)
+		)
+	)
 	(text "=3.3V"
 		(exclude_from_sim no)
@@
 			)
 			(justify left bottom)
+		)
+	)
+	(text "TODO: works only in one orientation"
+		(exclude_from_sim no)
+		(at 72.39 194.31 0)
+		(effects
+			(font
+				(size 1.27 1.27)
+			)
 		)
 	)
@@
 		)
 	)
+	(text "TODO: missing caps on TX"
+		(exclude_from_sim no)
+		(at 435.61 182.88 0)
+		(effects
+			(font
+				(size 1.27 1.27)
+			)
+		)
+	)

Commit message: WIP ports-two redesign
Parts:
- removed D2, D3: PMEG1020EA,115, Diode_SMD:D_SOD-323, symbol Device:D_Schottky_Small_Filled
- removed FB1, FB2: 220@100MHz 1.4A, Inductor_SMD:L_0603_1608Metric, symbol Device:FerriteBead_Small
- removed J7: Conn_01x04, Connector_JST:JST_SH_SM04B-SRSS-TB_1x04-1MP_P1.00mm_Horizontal, symbol Connector_Generic:Conn_01x04
- removed R39, R40, R43, R44: 22k, Resistor_SMD:R_0402_1005Metric, symbol Device:R_Small
- removed U12, U13: LM2830XQMFE/NOPB, Package_TO_SOT_SMD:SOT-23-5, symbol pocket-reform:LM2830XQMFE
- removed U2: HD3SS3220IRNHT, footprints:QFN40P450X250X80-31N120X320, symbol HD3SS3220IRNHT:HD3SS3220IRNHT
- added C44, C45, C46, C47, C52, C55, C56, C57, C58, C59: 0.1uF, Capacitor_SMD:C_0402_1005Metric, symbol Device:C_Small
- added C48, C49, C53, C54: 1uF, Capacitor_SMD:C_0402_1005Metric, symbol Device:C_Small
- added C50, C51: 4.7uF, Capacitor_SMD:C_0402_1005Metric, symbol Device:C_Small
- added FB5, FB6: 100@100MHz 3A, Inductor_SMD:L_0402_1005Metric, symbol Device:FerriteBead_Small
- added J8: Conn_01x12_Pin, Connector_FFC-FPC:Hirose_FH12-12S-0.5SH_1x12-1MP_P0.50mm_Horizontal, symbol Connector:Conn_01x12_Pin
- added R10, R20: 0, Resistor_SMD:R_0402_1005Metric, symbol Device:R_Small
- added R19: 900k, Resistor_SMD:R_0402_1005Metric, symbol Device:R_Small
- added TP3, TP4, TP5, TP6, TP7: TestPoint, TestPoint:TestPoint_Pad_D1.0mm, symbol Connector:TestPoint
- added U12, U13: TLV62569DBV, Package_TO_SOT_SMD:SOT-23-5, symbol Regulator_Switching:TLV62569DBV
- added U14: EQCO5X31C0-I_6NX, footprints:QFN50P400X400X100-21N-D, symbol EQCO5X31C0-I_6NX:EQCO5X31C0-I_6NX
- added U15: LP5907MFX-1.2, Package_TO_SOT_SMD:SOT-23-5, symbol Regulator_Linear:LP5907MFX-1.2
- added U16, U18: TUSB321, Package_DFN_QFN:Texas_X2QFN-12_1.6x1.6mm_P0.4mm, symbol Interface_USB:TUSB321
- added U17, U2: TMUXHS4212, footprints:Texas-VQFN20_2.5x4.5mm_RKS, symbol reform-camera:TMUXHS4212
- C17: value 47uF -> 0.1uF; footprint Capacitor_SMD:C_1206_3216Metric -> Capacitor_SMD:C_0402_1005Metric; LCSC (none) -> C1525; Manufacturer TDK -> Samsung; Manufacturer_No C3216X5R1E476M160AC -> CL05B104KO5NNNC
- C18: LCSC (none) -> C1525
- J1, J2: footprint footprints:MOLEX_105450-0101 -> Connector_USB:USB_C_Receptacle_Molex_105450-0101
- J5: footprint Connector_FFC-FPC:Hirose_FH12-20S-0.5SH_1x20-1MP_P0.50mm_Horizontal -> footprints:AMPHENOL_SFV20R-2STE1HLF; Manufacturer Hirose -> Amphenol ICC; Manufacturer_No FH12-20S-0.5SH(55) -> SFV20R-2STE1HLF
- R11: value 10k -> 0; LCSC (none) -> C242160; Manufacturer Yageo -> Panasonic; Manufacturer_No RC0402FR-7D10KL -> ERJ2GE0R00X
- R12: value 909k -> 10k; LCSC (none) -> C242160; Manufacturer Bourns -> Panasonic; Manufacturer_No CR0402-FX-9093GLF -> ERJ2GE0R00X
- R13, R22: value 200k -> 10k; Manufacturer Bourns -> Yageo; Manufacturer_No CR0402-JW-204GLF -> RC0402FR-7D10KL
- R14: value 0 -> 4.7k; Manufacturer Vishay Dale -> Yageo; Manufacturer_No CRCW04020000Z0EDC -> RC0402FR-7D10KL
- R15: value 0 -> 900k; Manufacturer Vishay Dale -> (none); Manufacturer_No CRCW04020000Z0EDC -> (none)
- R16, R17, R21: LCSC (none) -> C242160; Manufacturer Vishay Dale -> Panasonic; Manufacturer_No CRCW04020000Z0EDC -> ERJ2GE0R00X
- R18: value 200k -> 0; LCSC (none) -> C242160; Manufacturer Bourns -> Panasonic; Manufacturer_No CR0402-JW-204GLF -> ERJ2GE0R00X
- R23: value 200k -> 4.7k; Manufacturer Bourns -> Yageo; Manufacturer_No CR0402-JW-204GLF -> RC0402FR-7D10KL
- R24: value 200k -> 0; Manufacturer Bourns -> Vishay Dale; Manufacturer_No CR0402-JW-204GLF -> CRCW04020000Z0EDC
- R31: value 100k -> 10k; Manufacturer_No RC0402FR-07100KL -> (none)
- R35, R36: value 100k -> 10k
- TP1, TP2: footprint TestPoint:TestPoint_Pad_1.0x1.0mm -> TestPoint:TestPoint_Pad_D1.0mm; Manufacturer DNP -> (none); Manufacturer_No DNP -> (none); now fitted
Connections:
- net +1V1: now also R25.1
- net +3V3: now also R11.2, R12.2, R16.2, R24.1, C49.1, U15.1 (IN); no longer R21.2
- net +5V: now also C18.1, R13.1, R14.1, R15.1, R22.1, R23.1, C45.1, J8.10 (Pin_10), J8.11 (Pin_11), R19.1, U12.4 (VIN), U13.4 (VIN), U16.12 (VDD), U18.12 (VDD); no longer R25.2
- net GND: now also J5.13 (Pin_13), J5.3 (Pin_3), J5.6 (Pin_6), C44.2, C45.2, C48.2, C49.2, C52.2, C53.2, C54.2, C55.2, J8.12 (Pin_12), J8.3 (Pin_3), J8.6 (Pin_6), J8.9 (Pin_9), R10.2, U12.2 (GND), U13.2 (GND), U14.1 (GND_1), U14.21 (GND_2), U15.2 (GND), U16.10 (GND), U17.11 (GND), U17.20 (GND), U17.5 (GND), U17.PAD (GND), U18.10 (GND), U2.11 (GND), U2.20 (GND), U2.5 (GND), U2.PAD (GND); no longer J5.15 (Pin_15), J5.18 (Pin_18), J5.8 (Pin_8), R16.1, R17.1
- net HDMI_CEC: now also J5.14 (Pin_14); no longer J5.7 (Pin_7)
- net HDMI_CLKN: now also J5.11 (Pin_11); no longer J5.10 (Pin_10)
- net HDMI_CLKP: now also J5.10 (Pin_10); no longer J5.11 (Pin_11)
- net HDMI_HPD: now also J5.17 (Pin_17); no longer J5.4 (Pin_4)
- net HDMI_SCL: now also J5.15 (Pin_15); no longer J5.5 (Pin_5)
- net HDMI_SDA: now also J5.16 (Pin_16); no longer J5.6 (Pin_6)
- net HDMI_TX0N: now also J5.8 (Pin_8); no longer J5.13 (Pin_13)
- net HDMI_TX0P: now also J5.7 (Pin_7); no longer J5.14 (Pin_14)
- net HDMI_TX1N: now also J5.5 (Pin_5); no longer J5.16 (Pin_16)
- net HDMI_TX1P: now also J5.4 (Pin_4); no longer J5.17 (Pin_17)
- net HDMI_TX2N: now also J5.2 (Pin_2); no longer J5.19 (Pin_19)
- net HDMI_TX2P: now also J5.1 (Pin_1); no longer J5.20 (Pin_20)
- net MUX_3V3: now also C17.1, R11.1, R16.1, C44.1, U17.6 (VCC), U2.6 (VCC); no longer C18.1, R18.2, R21.1
- net USB2_RXN: now also C59.1; no longer U1.56 (USB_SSTXM_UP)
- net USB2_RXP: now also C58.1; no longer U1.55 (USB_SSTXP_UP)
- net USB2_TXN: now also U14.13 (SDBIN); no longer U1.59 (USB_SSRXM_UP)
- net USB2_TXP: now also U14.12 (SDBIP); no longer U1.58 (USB_SSRXP_UP)
- net USBH_1V1: now also R25.2
- net USBH_3V3: now also R24.2
- net USBH_3_DN: now also U1.10 (USB_DM_DN2), U9.2 (IO2), U9.9 (IO2); no longer U1.18 (USB_DM_DN3), U9.1 (IO1), U9.10 (IO1)
- net USBH_3_DP: now also U1.9 (USB_DP_DN2), U9.1 (IO1), U9.10 (IO1); no longer U1.17 (USB_DP_DN3), U9.2 (IO2), U9.9 (IO2)
- net USBH_4_DN: now also J8.1 (Pin_1)
- net USBH_4_DP: now also J8.2 (Pin_2)
- net USBC2_MUX_DIR: now reaches R18.1
- net USBC2_MUX_DIR: now also U18.11 (DIR)
- net at R36.2: now also U13.1 (EN)
- net at R41.2, R42.1: now also U13.5 (FB)
- net at L2.1: now also U13.3 (SW)
- net at L1.1: now also U12.3 (SW)
- net at R14.2: now also U16.4 (PORT)
- net at R17.2: now also U17.2 (~{OE})
- net at R15.2: now also U16.5 (VBUS_DET)
- net at TP2.1: now also U16.6 (~{VCONN_FAULT})
- net at TP1.1: now also U16.9 (ID)
- net at R13.2: now also U16.3 (CURRENT_MODE)
- net at R37.2, R38.1: now also U12.5 (FB)
- net at R35.2: now also U12.1 (EN)
- net CC1 renamed USBC1_CC1
- net USBC1_CC1: now also U16.1 (CC1)
- net CC2 renamed USBC1_CC2
- net USBC1_CC2: now also U16.2 (CC2)
- net MUXCC1 renamed USBC2_CC1
- net USBC2_CC1: now also U18.1 (CC1); no longer R15.1
- net MUXCC2 renamed USBC2_CC2
- net USBC2_CC2: now also U18.2 (CC2); no longer R14.1
- removed net MUX_5V: C17.1, R11.1, R12.1, R13.1, R22.2, R23.2, R24.2, R25.1
- net USB3_1_SSTXCN renamed USBH3_TXCN
- net USB3_1_SSTXCP renamed USBH3_TXCP
- net USBH_1A_AC_TXN renamed USBC2A_TXCN
- net USBH_1A_AC_TXP renamed USBC2A_TXCP
- net USBH_1A_RXN renamed USBH3_RXN
- net USBH3_RXN: now also U1.15 (USB_SSRXM_DN2); no longer U1.7 (USB_SSRXM_DN1)
- net USBH_1A_RXP renamed USBH3_RXP
- net USBH3_RXP: now also U1.14 (USB_SSRXP_DN2); no longer U1.6 (USB_SSRXP_DN1)
- net USBH_1A_TXN renamed USBH1_TXN
- net USBH1_TXN: now also U2.7 (A1_P); no longer C34.1
- net USBH_1A_TXP renamed USBH1_TXP
- net USBH1_TXP: now also U2.8 (A1_N); no longer C36.1
- net USBH_1B_AC_TXN renamed USBC2B_TXCN
- net USBH_1B_AC_TXP renamed USBC2B_TXCP
- net USBH_1B_RXN renamed USBH4_RXN
- net USBH4_RXN: now also J8.7 (Pin_7)
- net USBH_1B_RXP renamed USBH4_RXP
- net USBH4_RXP: now also J8.8 (Pin_8)
- net USBH_1B_TXN renamed USBH4_TXP
- net USBH4_TXP: now also J8.5 (Pin_5)
- net USBH_1B_TXP renamed USBH4_TXN
- net USBH4_TXN: now also J8.4 (Pin_4)
- net USBH_1_DN renamed USBC2_DN
- net USBC2_DN: now also U1.18 (USB_DM_DN3); no longer U1.2 (USB_DM_DN1)
- net USBH_1_DP renamed USBC2_DP
- net USBC2_DP: now also U1.17 (USB_DP_DN3); no longer U1.1 (USB_DP_DN1)
- net USBH_2A_AC_TXN renamed USBC1A_TXCN
- net USBH_2A_AC_TXP renamed USBC1A_TXCP
- net USBH_2A_RXN renamed USBC1A_RXN
- net USBC1A_RXN: now also U2.18 (B0_N); no longer U1.15 (USB_SSRXM_DN2)
- net USBH_2A_RXP renamed USBC1A_RXP
- net USBC1A_RXP: now also U2.19 (B0_P); no longer U1.14 (USB_SSRXP_DN2)
- net USBH_2A_TXN renamed USBC1A_TXN
- net USBC1A_TXN: now also U2.16 (B1_N); no longer U1.12 (USB_SSTXM_DN2)
- net USBH_2A_TXP renamed USBC1A_TXP
- net USBC1A_TXP: now also U2.17 (B1_P); no longer U1.11 (USB_SSTXP_DN2)
- net USBH_2B_AC_TXN renamed USBC1B_TXCN
- net USBH_2B_AC_TXP renamed USBC1B_TXCP
- net USBH_2B_RXN renamed USBC1B_RXN
- net USBC1B_RXN: now also U2.15 (C0_P); no longer U1.22 (USB_SSRXP_DN3)
- net USBH_2B_RXP renamed USBC1B_RXP
- net USBC1B_RXP: now also U2.14 (C0_N); no longer U1.23 (USB_SSRXM_DN3)
- net USBH_2B_TXN renamed USBC1B_TXN
- net USBC1B_TXN: now also U2.13 (C1_P); no longer U1.20 (USB_SSTXM_DN3)
- net USBH_2B_TXP renamed USBC1B_TXP
- net USBC1B_TXP: now also U2.12 (C1_N); no longer U1.19 (USB_SSTXP_DN3)
- net USBH_2_DN renamed USBC1_DN
- net USBC1_DN: now also U1.2 (USB_DM_DN1); no longer U1.10 (USB_DM_DN2)
- net USBH_2_DP renamed USBC1_DP
- net USBC1_DP: now also U1.1 (USB_DP_DN1); no longer U1.9 (USB_DP_DN2)
- net USBH_MUXA_RXN renamed USBC2A_RXN
- net USBC2A_RXN: now also U17.18 (B0_N)
- net USBH_MUXA_RXP renamed USBC2A_RXP
- net USBC2A_RXP: now also U17.19 (B0_P)
- net USBH_MUXA_TXN renamed USBC2A_TXN
- net USBC2A_TXN: now also U17.16 (B1_N)
- net USBH_MUXA_TXP renamed USBC2A_TXP
- net USBC2A_TXP: now also U17.17 (B1_P)
- net USBH_MUXB_RXN renamed USBC2B_RXN
- net USBC2B_RXN: now also U17.15 (C0_P)
- net USBH_MUXB_RXP renamed USBC2B_RXP
- net USBC2B_RXP: now also U17.14 (C0_N)
- net USBH_MUXB_TXN renamed USBC2B_TXN
- net USBC2B_TXN: now also U17.13 (C1_P)
- net USBH_MUXB_TXP renamed USBC2B_TXP
- net USBC2B_TXP: now also U17.12 (C1_N)
- new net: R22.2, U18.3 (CURRENT_MODE)
- new net: R23.2, U18.4 (PORT)
- new net: R19.2, U18.5 (VBUS_DET)
- new net: TP3.1, U18.6 (~{VCONN_FAULT})
- new net: TP7.1, U18.9 (ID)
- new net: R20.2, U2.2 (~{OE})
- new net: R21.2, U2.9 (SEL)
- new net: R18.2, U17.9 (SEL)
- new net: TP4.1, U14.7 (TSC)
- new net: TP5.1, U14.10 (TSI)
- new net: J5.18 (Pin_18), J5.19 (Pin_19), J5.20 (Pin_20), R1.1
- new net: C50.1, FB5.1, U14.5 (PLLA1)
- new net: C51.1, U14.16 (PLLB2)
- new net: C51.2, FB6.2, U14.15 (PLLB1)
- new net: R10.1, U14.20 (TEST0)
- new net: R12.1, U15.3 (EN)
- new net: C50.2, U14.6 (PLLA2)
- new net: TP6.1, U14.11 (LOM)
- new net +1V2: C48.1, C52.1, C53.1, C54.1, C55.1, FB5.2, FB6.1, U14.14 (VCCB), U14.4 (VCCA), U15.5 (OUT)
- new net SDAON: C58.2, U14.9 (SDAON)
- new net SDAOP: C59.2, U14.8 (SDAOP)
- new net SDBON: C56.1, U14.19 (SDBON)
- new net SDBOP: C57.1, U14.18 (SDBOP)
- new net UP_SSTXN: C47.2, U1.56 (USB_SSTXM_UP)
- new net UP_SSTXP: C46.2, U1.55 (USB_SSTXP_UP)
- new net USB2_RE_RXN: C46.1, U14.3 (SDAIN)
- new net USB2_RE_RXP: C47.1, U14.2 (SDAIP)
- new net USB2_RE_TXN: C56.2, U1.58 (USB_SSRXP_UP)
- new net USB2_RE_TXP: C57.2, U1.59 (USB_SSRXM_UP)
- new net USBC1_MUX_DIR: R21.1, U16.11 (DIR)
- new net USBH1_RXN: U1.7 (USB_SSRXM_DN1), U2.3 (A0_P)
- new net USBH1_RXP: U1.6 (USB_SSRXP_DN1), U2.4 (A0_N)
- new net USBH2_RXN: U1.23 (USB_SSRXM_DN3), U17.3 (A0_P)
- new net USBH2_RXP: U1.22 (USB_SSRXP_DN3), U17.4 (A0_N)
- new net USBH2_TXN: U1.20 (USB_SSTXM_DN3), U17.7 (A1_P)
- new net USBH2_TXP: U1.19 (USB_SSTXP_DN3), U17.8 (A1_N)
- new net USBH3_TXN: C34.1, U1.12 (USB_SSTXM_DN2)
- new net USBH3_TXP: C36.1, U1.11 (USB_SSTXP_DN2)
- new net ~{USB_MUX_OE}: R17.1, R20.1
- no-connect marks 20 -> 25
Other:
- note added: "HDMI"
- note added: "HDMI to port farm (flipped, top side)"
- note added: "NOTE: changed to 10k"
- note added: "TODO: 220nF?!"
- note added: "TODO: 5v inrush!"
- note added: "TODO: OE pulldown!"
- note added: "TODO: capacitor calc"
- note added: "TODO: caps check?"
- note added: "TODO: control reset via sysctl"
- note added: "TODO: double check resistors, L, EN pull"
- note added: "TODO: possibly 0R"
- note added: "TODO: wire up MUX_OE!"
- note added: "USB 3 Redriver"
- note added: "USB to camera"
- note added: "USB-C Data Mux 1"
- note added: "USB-C Data Mux 2"
- note added: "flipped in D-1"
- note added: "pair swapped on purpose!"
- note added: "pol. swap"
- note added: "pol. swap!"
- note added: "pol. swapped"
- note removed: "HDMI to port farm (flipped)"
- note removed: "TODO/FIXME: sda/scl flipped vs rcore+hdmiedp!"
- note removed: "TODO: DNP @ 22k"
- note removed: "TODO: change to 10k!"
- note removed: "TODO: double check ENN_CC, PORT"
- note removed: "TODO: flipped!"
- note removed: "TODO: missing caps on TX"
- note removed: "TODO: works only in one orientation"
- note removed: "https://www.ti.com/lit/ds/symlink/hd3ss3220.pdf?ts=1718344395887"
- moved on the sheet: C19, C20, C21, C22, C23, C24, C25, C26, C27, C28, C29, C30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
