File: nref-ports-two/nref-ports-two.kicad_sch (KiCad schematic)
At the start: 140 parts, among them J1 USB_C_Receptacle, J2 USB_C_Receptacle, J3 USB3_A, J4 HD0919MSMTTR, J5 Conn_01x20, J6 Conn_01x12_Pin, J8 Conn_01x12_Pin, U1 TUSB8041, U10 TPD4E02B04DQA, U11 TPD12S521, U12 TLV62569DBV, U13 TLV62569DBV, U14 EQCO5X31C0-I_6NX, U15 LP5907MFX-1.2, U16 TUSB321, U17 TMUXHS4212, U18 TUSB321, U2 TMUXHS4212, U3 TPD4E02B04DQA, U4 TPD4E02B04DQA, U5 TPD4E02B04DQA, U6 TPD4E02B04DQA, U7 TPD4E02B04DQA, U8 TPD4E02B04DQA, U9 TPD4E02B04DQA, Y1 24MHz

Commit message: ports-two: more routing
Connections:
- net USBC1A_RXN: now also U2.15 (C0_P); no longer U2.18 (B0_N)
- net USBC1A_RXP: now also U2.14 (C0_N); no longer U2.19 (B0_P)
- net USBC1A_TXN: now also U2.13 (C1_P); no longer U2.16 (B1_N)
- net USBC1A_TXP: now also U2.12 (C1_N); no longer U2.17 (B1_P)
- net USBC1B_RXN: now also U2.18 (B0_N), U5.4 (IO3), U5.7 (IO3); no longer U2.15 (C0_P), U5.1 (IO1), U5.10 (IO1)
- net USBC1B_RXP: now also U2.19 (B0_P), U5.5 (IO4), U5.6 (IO4); no longer U2.14 (C0_N), U5.2 (IO2), U5.9 (IO2)
- net USBC1B_TXCN: now also U5.1 (IO1), U5.10 (IO1); no longer U5.5 (IO4), U5.6 (IO4)
- net USBC1B_TXCP: now also U5.2 (IO2), U5.9 (IO2); no longer U5.4 (IO3), U5.7 (IO3)
- net USBC1B_TXN: now also U2.16 (B1_N); no longer U2.13 (C1_P)
- net USBC1B_TXP: now also U2.17 (B1_P); no longer U2.12 (C1_N)
- net USBC2A_RXN: now also U17.15 (C0_P); no longer U17.18 (B0_N)
- net USBC2A_RXP: now also U17.14 (C0_N); no longer U17.19 (B0_P)
- net USBC2A_TXN: now also U17.13 (C1_P); no longer U17.16 (B1_N)
- net USBC2A_TXP: now also U17.12 (C1_N); no longer U17.17 (B1_P)
- net USBC2B_RXN: now also U17.18 (B0_N), U8.4 (IO3), U8.7 (IO3); no longer U17.15 (C0_P), U8.1 (IO1), U8.10 (IO1)
- net USBC2B_RXP: now also U17.19 (B0_P), U8.5 (IO4), U8.6 (IO4); no longer U17.14 (C0_N), U8.2 (IO2), U8.9 (IO2)
- net USBC2B_TXCN: now also U8.1 (IO1), U8.10 (IO1); no longer U8.4 (IO3), U8.7 (IO3)
- net USBC2B_TXCP: now also U8.2 (IO2), U8.9 (IO2); no longer U8.5 (IO4), U8.6 (IO4)
- net USBC2B_TXN: now also U17.16 (B1_N); no longer U17.13 (C1_P)
- net USBC2B_TXP: now also U17.17 (B1_P); no longer U17.12 (C1_N)
- net MUX_3V3: no longer names the net of C17.1, R11.1, U2.6 (VCC)
- net MUX_3V3: no longer C44.1, R16.1, U17.6 (VCC)
- new net: C44.1, R16.1, U17.6 (VCC)
Other:
- note added: "- if SEL high"
- note added: "- if SEL low"
- note added: "NOTE: caps on USB2_TXN/P? no, TX caps are on RCORE"
- note added: "TODO: Rs on CC lines for swapping?"
- note added: "pol. swapped on purpose!"
- note removed: "pair swapped on purpose!"

Commit message: commit various notes / polishing for ports-one and ports-two
Parts:
- added R39, R40, R43: 0, Resistor_SMD:R_0402_1005Metric, symbol Device:R_Small
- C1, C2: LCSC (none) -> C1549
- C10, C11, C13, C14, C15, C21, C22, C23, C24, C27, C28, C29, C3, C30, C33, C34, C35, C36, C37, C38, C4, C46, C47, C5, C56, C57, C58, C59, C6, C7, C8, C9: LCSC (none) -> C307331
- C12, C16, C43: LCSC (none) -> C96446
- C17, C18, C44, C45, C52, C55: LCSC C1525 -> C307331
- C19, C20, C25, C26, C31, C32, C40, C42: LCSC (none) -> C96123
- C39, C41: LCSC (none) -> C59461
- C48, C49, C53, C54: LCSC C1525 -> C52923
- C50, C51: LCSC C307423 -> C23733
- D1: LCSC (none) -> C143772
- FB5, FB6: LCSC C14709 -> C124089; Manufacturer Murata -> FH; Manufacturer_No BLM18PG121SN1D -> CBW100505U101T
- J1, J2: LCSC (none) -> C134092
- J3: Notes (none) -> expensive, global sourcing
- J4: Manufacturer CUI -> Same Sky; Notes (none) -> unknown @ jlc
- J5: LCSC (none) -> C599468; Notes (none) -> low stock
- J6, J8: LCSC (none) -> C262661; Notes (none) -> jushuo
- L1: LCSC (none) -> C29780744; Manufacturer Murata -> cijang; Manufacturer_No DFE32CAH3R3MR0L -> FPB322520D-3R3MT0
- L2: LCSC (none) -> C5832378; Manufacturer Murata -> cijang; Manufacturer_No DFE32CAH3R3MR0L -> FTC322512SR22MBCA
- R1, R24, R25: LCSC (none) -> C17168; Manufacturer Vishay Dale -> Panasonic; Manufacturer_No CRCW04020000Z0EDC -> ERJ2GE0R00X
- R10, R11, R16, R18, R21: LCSC C242160 -> C17168
- R12: LCSC C242160 -> C25744; Manufacturer Panasonic -> Yageo; Manufacturer_No ERJ2GE0R00X -> RC0402FR-7D10KL
- R13, R22, R26, R30, R38, R42, R6: LCSC (none) -> C25744
- R14, R23: LCSC (none) -> C25900; Manufacturer_No RC0402FR-7D10KL -> RC0402FR-074K7L
- R15, R19: value 900k -> 909k; LCSC (none) -> C25799; Manufacturer (none) -> Uni-Royal; Manufacturer_No (none) -> 0402WGF9093TCE
- R17, R20: value 0 -> 10k; LCSC C242160 -> C25744; Manufacturer Panasonic -> Yageo; Manufacturer_No ERJ2GE0R00X -> RC0402FR-7D10KL
- R2, R3: LCSC (none) -> C26083
- R27, R29, R5, R8, R9: LCSC (none) -> C25900
- R28: LCSC (none) -> C25771
- R31: LCSC (none) -> C25744; Manufacturer_No (none) -> RC0402FR-7D10KL
- R32, R33, R34: LCSC (none) -> C25792
- R35, R36: LCSC (none) -> C25744; Manufacturer_No RC0402FR-07100KL -> RC0402FR-7D10KL
- R37: LCSC (none) -> C5126132
- R4: LCSC (none) -> C163452
- R41: LCSC (none) -> C2933099
- R7: LCSC (none) -> C96273
- TP1, TP2, TP3, TP7: now not fitted
- U1: LCSC (none) -> C544686; Manufacturer_No TUSB8041 -> TUSB8041IRGCR; Notes (none) -> alternative PNs
- U10, U3, U4, U5, U6, U7, U8, U9: LCSC (none) -> C2841426; Notes (none) -> clone
- U11: LCSC (none) -> C126920; Manufacturer_No TPD12S521 -> TPD12S521DBTR
- U12, U13: LCSC (none) -> C141836; Manufacturer (none) -> Texas Instruments; Manufacturer_No (none) -> TLV62569DBV
- U14: Height 1 -> (none); Manufacturer_Name Microchip -> (none); Manufacturer_Part_Number EQCO5X31C0-I/6NX -> (none); Mouser Part Number 494-EQCO5X31C0-I/6NX -> (none)
- U16, U18: LCSC (none) -> C2674046; Manufacturer (none) -> Texas Instruments; Manufacturer_No (none) -> TUSB321AI
- U17, U2: MPN TMUXHS4212RKSR -> (none)
- Y1: LCSC (none) -> C91744
Connections:
- net +5V: now also J5.18 (Pin_18), J5.19 (Pin_19), J5.20 (Pin_20); no longer R1.2
- net GND: now also R17.2, R20.1
- net USBC1_CC1: now also R1.1; no longer U16.1 (CC1)
- net USBC1_CC2: now also R39.1; no longer U16.2 (CC2)
- net USBC2_CC1: now also R40.1; no longer U18.1 (CC1)
- net USBC2_CC2: now also R43.1; no longer U18.2 (CC2)
- net at U17.2 (~{OE}): now also R17.1; no longer R17.2
- removed net ~{USB_MUX_OE}: R17.1, R20.1
- new net: R40.2, U18.1 (CC1)
- new net: R43.2, U18.2 (CC2)
- new net: R1.2, U16.1 (CC1)
- new net: R39.2, U16.2 (CC2)
Other:
- note removed: "TODO: 220nF?!"
- note removed: "TODO: 5v inrush!"
- note removed: "TODO: OE pulldown!"
- note removed: "TODO: Rs on CC lines for swapping?"
- note removed: "TODO: wire up MUX_OE!"
- company: (none) -> MNT Research GmbH
- title: (none) -> MNT Reform Next Port Board Two
- moved on the sheet: C45, C48, C49, C50, C51, C52, C53, C54, C55, C56, C57, C58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
Changed lines of the file:
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@@
 	(generator "eeschema")
 	(generator_version "9.0")
-	(paper "A2")
+	(paper "A1" portrait)
+	(title_block
+		(title "MNT Reform Next Port Board Two")
+		(date "2025-11-21")
+		(rev "D-2")
+		(company "MNT Research GmbH")
+		(comment 1 "Engineer: Lucie L. Hartmann")
+		(comment 2 "License: CERN OHL-S 2.0")
+		(comment 3 "https://mntre.com")
+	)

Commit message: ports-two: add TODOs after hw debugging
Other:
- note added: "> if the TUSB321 device is configured as a DFP and only ever used in DFP mode, the VBUS_DET pin can be left unconnected"
- note added: "TODO: capacitor calc. at least 120uF?!"
- note added: "TODO: caps missing!"
- note added: "TODO: pullup missing"
- note added: "TODO: pullups missing"
- note added: "TODO: remove"
- note added: "TODO: remove, we can't really source 3A"
- note added: "TODO: swap for TI"
- note removed: "TODO: caps check?"
- note removed: "TODO: six layer design, power close to diff pairs is questionable"

Commit message: PCBs: add various notes
Parts:
- added C60, C61: 0.1uF, Capacitor_SMD:C_0402_1005Metric, symbol Device:C_Small
- added R44, R45: 4.7k, Resistor_SMD:R_0402_1005Metric, symbol Device:R_Small
- R13, R15, R19, R22: now not fitted
Connections:
- net +3V3: now also R44.1, R45.1
- net USBC1_CC1: now also R39.1; no longer R1.1
- net USBC1_CC2: now also R1.1; no longer R39.1
- net USBC1_MUX_DIR: now also R45.2
- net USBC2_CC1: now also R43.1; no longer R40.1
- net USBC2_CC2: now also R40.1; no longer R43.1
- net USBC2_MUX_DIR: now also R44.2
- net USBH4_TXN: now also C61.2; no longer J8.4 (Pin_4)
- net USBH4_TXP: now also C60.2; no longer J8.5 (Pin_5)
- new net USBH4_AC_TXN: C61.1, J8.4 (Pin_4)
- new net USBH4_AC_TXP: C60.1, J8.5 (Pin_5)
Other:
- note added: "fixed: CCs needed to be swapped."
- note added: "fixed: tx caps were missing"
- note added: "we can't really source 3A"
- note removed: "TODO: caps missing!"
- note removed: "TODO: possibly 0R"
- note removed: "TODO: pullup missing"
- note removed: "TODO: remove"
- note removed: "TODO: remove, we can't really source 3A"
- note removed: "TODO: swap for TI"
- moved on the sheet: J8

Commit message: ports-two: snapshot of r2 before switch to nxp redriver
Parts:
- C10, C11, C13, C14, C15, C17, C18, C3, C33, C35, C37, C38, C4, C44, C45, C5, C52, C55, C6, C7, C8, C9: LCSC C307331 -> C1525
- C21, C22, C23, C24, C27, C28, C29, C30, C34, C36, C46, C47, C56, C57, C58, C59, C60, C61: value 0.1uF -> 0.22uF; LCSC C307331 -> C16772; Manufacturer_No CL05B104KO5NNNC -> CL05B224KO5NNNC
- J3: footprint footprints:WURTH_692121230100 -> footprints:USB-A-SMD_HC-USB3.0-C225-P; LCSC (none) -> C7501855; Manufacturer Wurth -> Hong Cheng; Manufacturer_No 692121230100 -> HC-USB3.0-C225-P; Notes expensive, global sourcing -> (none)
- J4: value HD0919MSMTTR -> A71-05H8-111N2; footprint footprints:HD0919MSMTTR -> footprints:HDMI-TH_A71-05H8-111N2; LCSC (none) -> C2880638; Manufacturer Same Sky -> XKB; Manufacturer_No HD09-19-MSMT-TR -> A71-05H8-111N2; Notes unknown @ jlc -> HD09-19-MSMT-TR alternative
- J5: footprint footprints:AMPHENOL_SFV20R-2STE1HLF -> footprints:FPC-SMD_AFC07-S20ECC-00; LCSC C599468 -> C11090; Manufacturer Amphenol ICC -> Jushuo; Manufacturer_No SFV20R-2STE1HLF -> AFC07-S20ECC-00; Notes low stock -> substitute: SFV20R-2STBE1HLF
Connections:
- net +5V: now also J5.1 (Pin_1), J5.2 (Pin_2), J5.3 (Pin_3); no longer J5.18 (Pin_18), J5.19 (Pin_19), J5.20 (Pin_20)
- net GND: now also J5.15 (Pin_15), J5.18 (Pin_18), J5.8 (Pin_8); no longer J5.13 (Pin_13), J5.3 (Pin_3), J5.6 (Pin_6)
- net HDMI_CEC: now also J5.7 (Pin_7); no longer J5.14 (Pin_14)
- net HDMI_CLKN: now also J5.10 (Pin_10); no longer J5.11 (Pin_11)
- net HDMI_CLKP: now also J5.11 (Pin_11); no longer J5.10 (Pin_10)
- net HDMI_HPD: now also J5.4 (Pin_4); no longer J5.17 (Pin_17)
- net HDMI_SCL: now also J5.6 (Pin_6); no longer J5.15 (Pin_15)
- net HDMI_SDA: now also J5.5 (Pin_5); no longer J5.16 (Pin_16)
- net HDMI_TX0N: now also J5.13 (Pin_13); no longer J5.8 (Pin_8)
- net HDMI_TX0P: now also J5.14 (Pin_14); no longer J5.7 (Pin_7)
- net HDMI_TX1N: now also J5.16 (Pin_16); no longer J5.5 (Pin_5)
- net HDMI_TX1P: now also J5.17 (Pin_17); no longer J5.4 (Pin_4)
- net HDMI_TX2N: now also J5.19 (Pin_19); no longer J5.2 (Pin_2)
- net HDMI_TX2P: now also J5.20 (Pin_20); no longer J5.1 (Pin_1)
- net USBH_3_DN: now also U9.1 (IO1), U9.10 (IO1); no longer U9.2 (IO2), U9.9 (IO2)
- net USBH_3_DP: now also U9.2 (IO2), U9.9 (IO2); no longer U9.1 (IO1), U9.10 (IO1)
Other:
- note added: "HDMI from MB (flipped, top side)"
- note added: "TODO: well, can't flip usb2 polarity!!"
- note added: "USB3 from MB (not flipped, bottom side)"
- note added: "pol. flipped"
- note removed: "HDMI to port farm (flipped, top side)"
- note removed: "TODO: pullups missing"
- note removed: "USB3 to port farm 2"
- moved on the sheet: J5
Changed lines of the file:
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@@
 (kicad_sch
-	(version 20250114)
+	(version 20260306)
 	(generator "eeschema")
-	(generator_version "9.0")
+	(generator_version "10.0")
 	(paper "A1" portrait)
 	(title_block
