File: nref-usb3-redriver/nref-usb3-redriver.kicad_pcb (KiCad board)
At the start: 4 copper layers, 54.5 x 32 mm, 41 parts, among them J2 Conn_01x12_Pin, J3 USB3_A, SW1 SW_DIP_x06, SW2 SW_DIP_x06, U1 TUSB522PIRGER, U10 TPD4E02B04DQA, U13 LM2830XQMFE/NOPB, U9 TPD4E02B04DQA

Commit message: add various notes in schematics
Routing:
- net GND: track 33.9 -> 34.4 mm, vias 98 -> 134
Other:
- board text added: "MNT RESEARCH 2025-08-27 USB3 REDRIVER TEST BOARD"
