File: nref-usb3-redriver/nref-usb3-redriver.kicad_sch (KiCad schematic)
At the start: 41 parts, among them J2 Conn_01x12_Pin, J3 USB3_A, SW1 SW_DIP_x06, SW2 SW_DIP_x06, U1 TUSB522PIRGER, U10 TPD4E02B04DQA, U13 LM2830XQMFE/NOPB, U9 TPD4E02B04DQA

Commit message: add various notes in schematics
Other:
- note added: "TODO: error: DN/DP flipped!"
Changed lines of the file:
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@@
+		)
+	)
+	(text "TODO: error: DN/DP flipped!"
+		(exclude_from_sim no)
+		(at 39.37 105.41 0)
+		(effects
+			(font
+				(size 1.27 1.27)
+			)
 		)
 	)
@@
 	)
 	(global_label "R_USB_RXN"
-		(shape input)
+		(shape output)
 		(at 318.77 82.55 0)
 		(fields_autoplaced yes)
@@
 	)
 	(global_label "R_USB_RXP"
-		(shape input)
+		(shape output)
 		(at 318.77 85.09 0)
 		(fields_autoplaced yes)
