File: nref-ports-one/nref-ports-one.kicad_sch (KiCad schematic)
At the start: 118 parts, among them J1 CONN_HEAD, J10 CONN_SPK, J2 DM3AT-SF-PEJM5, J3 09452812561, J4 USB_C_Receptacle, J5 Conn_01x10_Pin, J6 Conn_01x14_Pin, J7 Conn_01x12_Pin, J8 PWR, J9 Conn_01x10_Pin, U1 TPS7A0533PDBZ, U10 HD3SS3220IRNHT, U11 PCAL6416AHF, U12 TLV75518PDBV, U2 TLV320AIC3100, U3 TXS0108EPW, U4 SN74AVC1T45, U5 TPD4E02B04DQA, U6 TPD4E02B04DQA, U7 TPD4E02B04DQA, U8 FUSB302BMPX, U9 AP22815A

Commit message: ports-one: snapshot before d2
Other:
- note added: "TODO: smaller chip"
Changed lines of the file:
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@@
+		)
+	)
+	(text "TODO: smaller chip"
+		(exclude_from_sim no)
+		(at 331.47 165.1 0)
+		(effects
+			(font
+				(size 1.27 1.27)
+			)
 		)
 	)

Commit message: ports-one: WIP construction site
Other:
- note added: "TODO: replace with HD3SS460"
Changed lines of the file:
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@@
 		)
 	)
+	(text "TODO: replace with HD3SS460"
+		(exclude_from_sim no)
+		(at 74.93 209.55 0)
+		(effects
+			(font
+				(size 1.27 1.27)
+			)
+		)
+	)
 	(text "Sleeve"
 		(exclude_from_sim no)
@@
 			)
 		)
-		(property "Datasheet" ""
+		(property "Datasheet" "https://www.ti.com/lit/ds/symlink/hd3ss3220.pdf?ts=1718344395887"
 			(at 83.82 251.46 0)
 			(effects

Commit message: ports-one: schematics with new mux, local 5v, hard reset switch
Parts:
- removed D3: SS54, Diode_SMD:D_SMA, symbol Device:D_Schottky
- removed FB10: 100@100MHz 3A, Inductor_SMD:L_0603_1608Metric, symbol Device:FerriteBead_Small
- removed U10: HD3SS3220IRNHT, footprints:QFN40P450X250X80-31N120X320, symbol HD3SS3220IRNHT:HD3SS3220IRNHT
- removed U11: PCAL6416AHF, Package_DFN_QFN:HVQFN-24-1EP_4x4mm_P0.5mm_EP2.1x2.1mm, symbol Interface_Expansion:PCAL6416AHF
- removed U9: AP22815A, Package_TO_SOT_SMD:SOT-23-5, symbol reform2:AP22815
- added C45: 0.1uF, Capacitor_SMD:C_0402_1005Metric, symbol Device:C_Small
- added C46: 47uF, Capacitor_SMD:C_1210_3225Metric, symbol Device:C_Small
- added C47: 10uF, Capacitor_SMD:C_0603_1608Metric, symbol Device:C_Small
- added D3: LED_Red, LED_SMD:LED_0603_1608Metric, symbol Device:LED_Small
- added D4: LED_Blue, LED_SMD:LED_0603_1608Metric, symbol Device:LED_Small
- added J11: POWSW, Connector_JST:JST_SH_SM02B-SRSS-TB_1x02-1MP_P1.00mm_Horizontal, symbol Connector:Conn_01x02_Pin
- added L4: 6.8uH, Inductor_SMD:L_Taiyo-Yuden_NR-30xx, symbol Device:L
- added R36, R39, R41: 0, Resistor_SMD:R_0402_1005Metric, symbol Device:R_Small
- added R37: 13.7k, Resistor_SMD:R_0402_1005Metric, symbol Device:R_Small
- added R38: 10k, Resistor_SMD:R_0402_1005Metric, symbol Device:R_Small
- added R40: 0, Resistor_SMD:R_0603_1608Metric, symbol Device:R_Small
- added SW1: SW_Push, Button_Switch_SMD:SW_SPST_B3U-3000P, symbol Switch:SW_Push
- added TP1, TP2, TP3: TestPoint, TestPoint:TestPoint_Pad_D1.0mm, symbol Connector:TestPoint
- added U10: LMR51430, Package_TO_SOT_SMD:SOT-23-6, symbol Regulator_Switching:LMR51430
- added U11: TPS66021YBGR, footprints:YBG0028_TEX, symbol tps66021:TPS66021YBGR
- added U13: TMUXHS4212, footprints:Texas-VQFN20_2.5x4.5mm_RKS, symbol reform-camera:TMUXHS4212
- added U9: PCA9557BS, Package_DFN_QFN:HVQFN-16-1EP_3x3mm_P0.5mm_EP1.5x1.5mm, symbol Interface_Expansion:PCA9557BS
- C17, C21, C39, C40: footprint Capacitor_SMD:C_1206_3216Metric -> Capacitor_SMD:C_1210_3225Metric
- C38: value 47uF -> 0.1uF; footprint Capacitor_SMD:C_1206_3216Metric -> Capacitor_SMD:C_0402_1005Metric; LCSC (none) -> C1525; Manufacturer TDK -> Samsung; Manufacturer_No C3216X5R1E476M160AC -> CL05B104KO5NNNC
- C41: value 0.1uF -> 10uF; footprint Capacitor_SMD:C_0402_1005Metric -> Capacitor_SMD:C_0603_1608Metric; Manufacturer Samsung -> Yageo; Manufacturer_No CL05B104KO5NNNC -> CC0402KRX5R6BB105
- C8: value 0.1uF -> 1uF
- D1, D2: value LED_Small -> LED_Red
- J4: footprint footprints:MOLEX_105450-0101 -> Connector_USB:USB_C_Receptacle_Molex_105450-0101
- R22: now not fitted
- R23: value 200k -> 10k; LCSC C242160 -> C60490; Manufacturer Bourns -> Yageo; Manufacturer_No CR0402-JW-204GLF -> RC0402FR-7D10KL
- R25: value 200k -> 75k 1%; LCSC C242160 -> (none); Manufacturer Bourns -> (none); Manufacturer_No CR0402-JW-204GLF -> (none)
- R26: value 200k -> 0; Manufacturer Bourns -> Panasonic; Manufacturer_No CR0402-JW-204GLF -> ERJ2GE0R00X
- R27: value 200k -> 432k 1%; LCSC C242160 -> (none); Manufacturer Bourns -> (none); Manufacturer_No CR0402-JW-204GLF -> (none)
- R28: value 10k -> 20k 1%; LCSC C242160 -> (none); Manufacturer Yageo -> (none); Manufacturer_No RC0402FR-7D10KL -> (none)
- R29: value 909k -> 0; Manufacturer Bourns -> Panasonic; Manufacturer_No CR0402-FX-9093GLF -> ERJ2GE0R00X; now not fitted
- R30: value 200k -> 2.2k; LCSC C242160 -> C60490; Manufacturer Bourns -> Yageo; Manufacturer_No CR0402-JW-204GLF -> RC0402FR-7D10KL
- R31: value 0 -> 2.2k; LCSC C242160 -> C60490; Manufacturer Panasonic -> Yageo; Manufacturer_No ERJ2GE0R00X -> RC0402FR-7D10KL
- R32, R33: value 0 -> 1k; LCSC C242160 -> C60490; Manufacturer Panasonic -> Yageo; Manufacturer_No ERJ2GE0R00X -> RC0402FR-7D10KL
- R34: value 10k -> 0; LCSC C60491 -> C242160; Manufacturer Yageo -> Panasonic; Manufacturer_No RC0402FR-7D10KL -> ERJ2GE0R00X
- R35: value 0 -> 100k; LCSC C242160 -> (none); Manufacturer Panasonic -> (none); Manufacturer_No ERJ2GE0R00X -> (none)
Connections:
- net +3V3: now also R39.2, R41.2; no longer R22.2
- net +5V: no longer C32.1, C8.1, FB7.1, R19.2, R24.2, U1.3 (VI)
- net CC1: no longer R21.1
- net CC2: no longer R20.1
- net GND: now also R23.1, R25.2, R28.2, C45.2, C46.2, C47.2, R37.2, R38.2, U10.1 (GND), U11.B4 (GND), U13.11 (GND), U13.20 (GND), U13.5 (GND), U13.PAD (GND), U9.2 (A1), U9.3 (A2), U9.6 (VSS); no longer C38.2, R31.1, R35.1
- net MUX_3V3: now also R39.1, U13.6 (VCC); no longer R23.2
- net RP_FUSB_INT: now also TP3.1
- net RP_SCL0: now also U9.15 (SCL); no longer R32.2
- net RP_SDA0: now also U9.16 (SDA); no longer R33.2
- net STANDBY_3V3: now also R22.2, R29.1, R30.1, R31.1, R32.1, R33.1, C45.1, U9.14 (VDD); no longer C37.2, C41.1, R34.1, U8.3 (VDD), U8.4 (VDD)
- net USB1_RXN: now also U13.8 (A1_N)
- net USB1_RXP: now also U13.7 (A1_P)
- net USB1_TXN: now also U13.4 (A0_N)
- net USB1_TXP: now also U13.3 (A0_P)
- net USBH_2A_RXN: now also U13.16 (B1_N)
- net USBH_2A_RXP: now also U13.17 (B1_P)
- net USBH_2A_TXN: now also U13.14 (C0_N)
- net USBH_2A_TXP: now also U13.15 (C0_P)
- net USBH_2B_RXN: now also U13.12 (C1_N)
- net USBH_2B_RXP: now also U13.13 (C1_P)
- net USBH_2B_TXN: now also U13.18 (B0_N)
- net USBH_2B_TXP: now also U13.19 (B0_P)
- net USB_SRC_EN: now also R23.2, TP1.1, U11.A3 (EN1), U9.4 (IO0)
- net USB_VBUS: now also R27.2, U11.A2 (VBUS), U11.B2 (VBUS), U11.B3 (VBUS), U11.C2 (VBUS), U11.C3 (VBUS), U11.D2 (VBUS), U11.D3 (VBUS), U11.E2 (VBUS), U11.E3 (VBUS), U11.F2 (VBUS), U11.F3 (VBUS), U11.G2 (VBUS); no longer C40.1, R29.1, R30.1
- net VCC: now also C47.1, U10.3 (VIN)
- net VPD: now also C40.1, U11.B1 (PPHV), U11.C1 (PPHV), U11.D1 (PPHV), U11.E1 (PPHV), U11.F1 (PPHV)
- net at R25.1: now also U11.A4 (IREF)
- net at C28.1, C29.1, C30.1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: now also R41.1
- net at R30.2: now also U9.13 (~{RESET})
- net 5V_AUX: now reaches R26.1
- net 5V_AUX: now also FB7.1, R34.1, R35.1, C46.1, L4.2, R40.1
- net at R31.2: now also U9.1 (A0)
- net at U8.12 (VCONN): now also U8.13 (VCONN), R36.2
- net at R20.2: now also U13.2 (~{OE})
- net at R21.2: now also U13.9 (SEL)
- net at R27.1: now also R28.1, U11.F4 (OVP)
- net at R35.2: now also R37.1, U10.4 (FB)
- net LDO_3V3: now reaches R29.2
- net LDO_3V3: now also C37.2, R19.2, R24.1, U8.3 (VDD), U8.4 (VDD), R36.1
- net USB_SINK_EN: now reaches R19.1
- net USB_SINK_EN: now also TP2.1, U11.G1 (EN0), U9.5 (IO1)
- net at R34.2: now also C8.1, U1.3 (VI)
- removed net MUX_5V: C38.1, R24.1, R25.2, R26.2, R27.2, R28.1
- new net: C38.1, U10.6 (CB)
- new net: C38.2, L4.1, U10.2 (SW)
- new net: D3.1 (K), U9.10 (IO5)
- new net: D3.2 (A), R32.2
- new net: C32.1, R26.2, U11.G4 (VIN)
- new net: D4.1 (K), U9.11 (IO6)
- new net: D4.2 (A), R33.2
- new net: J11.1 (Pin_1), SW1.1
- new net: J11.2 (Pin_2), SW1.2
- new net: R40.2, U11.C4 (PP5V), U11.D4 (PP5V), U11.E4 (PP5V)
- new net: C41.1, R24.2, U11.G3 (VLDO)
- new net 5V_AUX_EN: R38.1, U10.5 (EN), U9.12 (IO7)
- new net USB_MUX_DIR: R21.1, U9.7 (IO2)
- new net ~{USB_FAULT}: U11.A1 (~{FLT}), U9.9 (IO4)
- new net ~{USB_MUX_OE}: R20.1, U9.8 (IO3)
- no-connect marks 28 -> 11
Other:
- note added: "GPIO bank controlled via I2C by System Controller"
- note added: "Local 5V for USB devices and speaker"
- note added: "NOTE: These +5V are currently unused"
- note added: "Standby Shutdown Switch"
- note added: "To/From USB-C connector"
- note added: "currently not connected"
- note added: "ix Industrial 10B-1"
- note removed: "GPIO bank controlled via I2C"
- note removed: "SOURCE"
- note removed: "TODO: 1uF input cap nominal"
- note removed: "TODO: Clamp"
- note removed: "TODO: VCONN"
- note removed: "TODO: WM8962B?"
- note removed: "TODO: backflow possible from standby to 3v3?"
- note removed: "TODO: double check ENN_CC, PORT"
- note removed: "TODO: possibly DNP"
- note removed: "TODO: pulldown missing on USB_SRC_EN!"
- note removed: "TODO: replace with HD3SS460"
- note removed: "TODO: resistor"
- note removed: "TODO: smaller chip"
- note removed: "TODO: these need larger footprints"
- note removed: "TODO: useful for low level peripherals?"
- note removed: "WARNING: do not use B version by accident (active low)"
- note removed: "https://www.ti.com/lit/ds/symlink/hd3ss3220.pdf?ts=1718344395887"
- note removed: "iX Industrial 10B-1"
- note removed: "rated to 28V"
- moved on the sheet: C26, C27, C28, C29, C30, C31, C37, C39, C40, C42, C43, C44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

Commit message: ports-one: add redriver, routing WIP
Parts:
- added U14: EQCO5X31C0-I_6NX, footprints:QFN50P400X400X100-21N-D, symbol EQCO5X31C0-I_6NX:EQCO5X31C0-I_6NX
Connections:
- net GND: now also U14.1 (GND_1), U14.21 (GND_2)
- net USB1_RXN: now also U14.9 (SDAON); no longer U13.8 (A1_N)
- net USB1_RXP: now also U14.8 (SDAOP); no longer U13.7 (A1_P)
- net USB1_TXN: now also U14.13 (SDBIN); no longer U13.4 (A0_N)
- net USB1_TXP: now also U14.12 (SDBIP); no longer U13.3 (A0_P)
- net USBH_2A_AC_TXN: now also U6.1 (IO1), U6.10 (IO1); no longer U6.4 (IO3), U6.7 (IO3)
- net USBH_2A_AC_TXP: now also U6.2 (IO2), U6.9 (IO2); no longer U6.5 (IO4), U6.6 (IO4)
- net USBH_2A_RXN: now also U13.18 (B0_N), U6.4 (IO3), U6.7 (IO3); no longer U13.16 (B1_N), U6.1 (IO1), U6.10 (IO1)
- net USBH_2A_RXP: now also U13.19 (B0_P), U6.5 (IO4), U6.6 (IO4); no longer U13.17 (B1_P), U6.2 (IO2), U6.9 (IO2)
- net USBH_2A_TXN: now also U13.12 (C1_N); no longer U13.14 (C0_N)
- net USBH_2A_TXP: now also U13.13 (C1_P); no longer U13.15 (C0_P)
- net USBH_2B_RXN: now also U13.14 (C0_N); no longer U13.12 (C1_N)
- net USBH_2B_RXP: now also U13.15 (C0_P); no longer U13.13 (C1_P)
- net USBH_2B_TXN: now also U13.16 (B1_N); no longer U13.18 (B0_N)
- net USBH_2B_TXP: now also U13.17 (B1_P); no longer U13.19 (B0_P)
- new net USB1_RE_RXN: U13.3 (A0_P), U14.3 (SDAIN)
- new net USB1_RE_RXP: U13.4 (A0_N), U14.2 (SDAIP)
- new net USB1_RE_TXN: U13.7 (A1_P), U14.19 (SDBON)
- new net USB1_RE_TXP: U13.8 (A1_N), U14.18 (SDBOP)
Other:
- note added: "Sysctl GPIO Bank"
- note added: "TODO"
- note added: "USB-C Data Mux"
- note added: "USB-C PD Power Mux"
- note added: "pair swapped on purpose!"

Commit message: ports-one: add redriver circuit
Parts:
- added C48, C49, C53, C54: 1uF, Capacitor_SMD:C_0402_1005Metric, symbol Device:C_Small
- added C50, C51: 4.7uF, Capacitor_SMD:C_0402_1005Metric, symbol Device:C_Small
- added C52, C55: 0.1uF, Capacitor_SMD:C_0402_1005Metric, symbol Device:C_Small
- added FB5, FB6: 100@100MHz 3A, Inductor_SMD:L_0603_1608Metric, symbol Device:FerriteBead_Small
- added R42, R43: 0, Resistor_SMD:R_0402_1005Metric, symbol Device:R_Small
- added TP4, TP5, TP6, TP7: TestPoint, TestPoint:TestPoint_Pad_D1.0mm, symbol Connector:TestPoint
- added U15: LP5907MFX-1.2, Package_SON:Texas_X2SON-4_1x1mm_P0.65mm, symbol Regulator_Linear:LP5907MFX-1.2
Connections:
- net +3V3: now also C49.1, R42.2, U15.1 (IN)
- net GND: now also C48.2, C49.2, C52.2, C53.2, C54.2, C55.2, R43.2, U15.2 (GND)
- net at U14.10 (TSI): now also TP5.1
- net at U14.11 (LOM): now also TP6.1
- net +1V2: now reaches U14.14 (VCCB)
- net +1V2: now also U14.4 (VCCA), C48.1, C52.1, C53.1, C54.1, C55.1, FB5.2, FB6.1, U15.5 (OUT)
- net at U14.15 (PLLB1): now also C51.2, FB6.2
- net at U14.16 (PLLB2): now also C51.1
- net at U14.20 (TEST0): now also R43.1, TP7.1
- net at U14.5 (PLLA1): now also C50.1, FB5.1
- net at U14.6 (PLLA2): now also C50.2
- net at U14.7 (TSC): now also TP4.1
- new net: R42.1, U15.3 (EN)
- no-connect marks 11 -> 12
Other:
- note added: "USB 3 Redriver"
- note removed: "TODO"
- moved on the sheet: C32, C40, C41, C42, R19, R20, R21, R22, R23, R24, R25, R26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

Commit message: ports-one: routing snapshot
Parts:
- removed R24: 0, Resistor_SMD:R_0402_1005Metric, symbol Device:R_Small
- FB1, FB2, FB3, FB4, FB5, FB6, FB7, FB8, FB9: footprint Inductor_SMD:L_0603_1608Metric -> Inductor_SMD:L_0402_1005Metric; Manufacturer_No BLM18PG121SN1D -> (none)
Connections:
- net LDO_3V3: now also C41.1, U11.G3 (VLDO)
- net USBH_2A_AC_TXN renamed USB_B_AC_TXN
- net USB_B_AC_TXN: now also U6.4 (IO3), U6.7 (IO3); no longer U6.1 (IO1), U6.10 (IO1)
- net USBH_2A_AC_TXP renamed USB_B_AC_TXP
- net USB_B_AC_TXP: now also U6.5 (IO4), U6.6 (IO4); no longer U6.2 (IO2), U6.9 (IO2)
- removed net USBH_2A_RXN: J4.B10 (RX1-), U13.18 (B0_N), U6.4 (IO3), U6.7 (IO3)
- removed net USBH_2A_RXP: J4.B11 (RX1+), U13.19 (B0_P), U6.5 (IO4), U6.6 (IO4)
- net USBH_2A_TXN renamed USB_B_TXN
- net USB_B_TXN: now also U13.13 (C1_P); no longer U13.12 (C1_N)
- net USBH_2A_TXP renamed USB_B_TXP
- net USB_B_TXP: now also U13.12 (C1_N); no longer U13.13 (C1_P)
- net USBH_2B_AC_TXN renamed USB_A_AC_TXN
- net USB_A_AC_TXN: now also U7.1 (IO1), U7.10 (IO1); no longer U7.4 (IO3), U7.7 (IO3)
- net USBH_2B_AC_TXP renamed USB_A_AC_TXP
- net USB_A_AC_TXP: now also U7.2 (IO2), U7.9 (IO2); no longer U7.5 (IO4), U7.6 (IO4)
- removed net USBH_2B_RXN: J4.A10 (RX2-), U13.14 (C0_N), U7.1 (IO1), U7.10 (IO1)
- removed net USBH_2B_RXP: J4.A11 (RX2+), U13.15 (C0_P), U7.2 (IO2), U7.9 (IO2)
- net USBH_2B_TXN renamed USB_A_TXN
- net USBH_2B_TXP renamed USB_A_TXP
- new net USB_A_RXN: J4.A10 (RX2-), U13.18 (B0_N), U7.4 (IO3), U7.7 (IO3)
- new net USB_A_RXP: J4.A11 (RX2+), U13.19 (B0_P), U7.5 (IO4), U7.6 (IO4)
- new net USB_B_RXN: J4.B10 (RX1-), U13.15 (C0_P), U6.1 (IO1), U6.10 (IO1)
- new net USB_B_RXP: J4.B11 (RX1+), U13.14 (C0_N), U6.2 (IO2), U6.9 (IO2)

Commit message: WIP nref-ports-one: routing done, 3d checks to do
Parts:
- removed FB1: 100@100MHz 3A, Inductor_SMD:L_0402_1005Metric, symbol Device:FerriteBead_Small
- removed FB2: DNP, Inductor_SMD:L_0402_1005Metric, symbol Device:FerriteBead_Small
- removed TP7: TestPoint, TestPoint:TestPoint_Pad_D1.0mm, symbol Connector:TestPoint
- added R24, R44: 0, Resistor_SMD:R_0402_1005Metric, symbol Device:R_Small
Connections:
- net GND: now also R24.1, R44.1; no longer C8.2, U1.1 (GND)
- net GNDA: now also C8.2, U1.1 (GND), R24.2, R44.2
