File: nref-ports-one/nref-ports-one.kicad_pcb (KiCad board)
At the start: 4 copper layers, 88 x 35.8 mm, 153 parts, among them J1 CONN_HEAD, J10 CONN_SPK, J11 POWSW, J12 SBU, J2 DM3AT-SF-PEJM5, J3 09452812561, J4 USB_C_Receptacle, J5 Conn_01x10_Pin, J6 Conn_01x14_Pin, J7 Conn_01x12_Pin, J8 PWR, J9 Conn_01x10_Pin, SW1 SW_Push, U1 TPS7A0533PDBZ, U10 LMR51430, U11 TPS66021YBGR, U12 TLV75518PDBV, U13 TMUXHS4212, U14 EQCO5X31C0-I_6NX, U15 LP5907MFX-1.2, U2 TLV320AIC3100, U3 TXS0108EPW, U4 SN74AVC1T45, U5 TPD4E02B04DQA, U6 TPD4E02B04DQA, U7 TPD4E02B04DQA, U8 FUSB302BMPX, U9 PCA9557RGVR

Commit message: ports left/one fixes
Parts:
- R45, R46: value 33 -> 0
- moved R46 20.7 mm to (124.5, 123.4), turned to 90 degrees
- moved R45 19.2 mm to (123.5, 123.4), turned to 90 degrees
- moved J12 8.81 mm to (108.8, 134.2), turned to 0 degrees
- moved C43 8.56 mm to (101.5, 126.0), turned to 180 degrees
- moved C44 8.48 mm to (105.2, 128.7)
- moved FB3 8.48 mm to (105.2, 126.8)
- moved U12 8.48 mm to (102.6, 128.3)
Connections:
- net Net-(J12-Pin_1) renamed /SBU_R_N
- net Net-(J12-Pin_2) renamed /SBU_R_P
Routing:
- net SBU_P: track 96.3 -> 71.4 mm
- net SBU_N: track 96.2 -> 71.5 mm
- net /SBU_R_N: track 8.28 -> 21.1 mm
- net /SBU_R_P: track 9.96 -> 20.6 mm
- net +1V8: track 48.7 -> 56.9 mm
- net +3V3: track 155.6 -> 160.7 mm
- net Net-(U2-DVDD): track 10.2 -> 13.3 mm
- net GND: track 73.0 -> 71.4 mm, vias 234 -> 231
- net GNDA: vias 44 -> 48
Other:
- board text removed: "TODO: caps might be too high"
