File: nref-flex/nref-flex-usb3-one/nref-flex-usb3-one.kicad_pcb (KiCad board)
At the start: 2 copper layers, 6.5 x 145.1 mm, 3 parts, among them J8 Conn_01x12_Pin, J9 Conn_01x12_Pin

Commit message: commit various flex changes
Parts:
- moved J9 9.90 mm to (71.8, 192.9)
Routing:
- net +5V: track 141.5 -> 154.5 mm, vias 2 -> 8
- net USB1_DN: track 141.4 -> 151.3 mm
- net USB1_TXN: track 141.4 -> 151.3 mm
- net USB1_RXN: track 141.4 -> 151.3 mm
- net USB1_DP: track 141.4 -> 151.3 mm
- net USB1_TXP: track 141.4 -> 151.3 mm
- net USB1_RXP: track 141.4 -> 151.3 mm
- net GND: track 160.6 -> 170.5 mm, vias 16 -> 70
Other:
- board size 6.5 x 145.1 mm -> 6.5 x 155 mm
- board text added: "50um dielectric, 50oz copper trace w: 0.1mm, spacing: 0.18mm target length: 155mm"
- board text added: "MNT Reform Next Internal USB3—155mm—Version 20251006"
- board text removed: "MNT Reform Next Internal USB3—145mm—Version 20250723"
- board text removed: "trace w: 0.13, spacing: 0.2 target length: 145mm"

Commit message: PCBs: add various notes
Parts:
- moved J9 10.0 mm to (71.8, 182.9)
Routing:
- net USB1_TXP: track 151.3 -> 141.3 mm
- net USB1_TXN: track 151.3 -> 141.3 mm
- net USB1_RXN: track 151.3 -> 141.3 mm
- net USB1_DP: track 151.3 -> 141.3 mm
- net USB1_DN: track 151.3 -> 141.3 mm
- net +5V: track 154.5 -> 144.5 mm
- net USB1_RXP: track 151.3 -> 141.3 mm
- net GND: track 170.5 -> 161.5 mm, vias 70 -> 67
Other:
- board size 6.5 x 155 mm -> 6.5 x 145 mm
- board text added: "50um dielectric, 50oz copper trace w: 0.1mm, spacing: 0.18mm target length: 145mm"
- board text added: "MNT Reform Next Internal USB3—145mm—Version 20251210"
- board text removed: "50um dielectric, 50oz copper trace w: 0.1mm, spacing: 0.18mm target length: 155mm"
- board text removed: "MNT Reform Next Internal USB3—155mm—Version 20251006"
