File: nref-batterypack-v3/nref-batterypack-backside.kicad_sch (KiCad schematic)
At the start: 8 parts, among them J1 C1+, J2 C2-, J3 C3+, J4 C4-, J5 FRONT_CONN

Commit message: batterypack v3 front+back pcbs polished for ordering
Parts:
- removed H2: MountingHole, MountingHole:MountingHole_2.2mm_M2, symbol Mechanical:MountingHole
- J1, J3: footprint footprints:S713145R -> footprints:S174146R; MPN (none) -> S174146R; Manufacturer (none) -> Harwin
- J2, J4: footprint footprints:S713145R -> footprints:S70332002045R; MPN (none) -> S70-332002045R; Manufacturer (none) -> Harwin
- J5: footprint Connector_JST:JST_SHL_SM02B-SHLS-TF_1x02-1MP_P1.00mm_Horizontal -> Connector_JST:JST_SH_SM02B-SRSS-TB_1x02-1MP_P1.00mm_Horizontal; MPN (none) -> SM02B-SRSS-TB; Manufacturer (none) -> JST
Changed lines of the file:
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@@
 			)
 		)
-		(property "Footprint" "footprints:S713145R"
+		(property "Footprint" "footprints:S70332002045R"
 			(at 106.68 96.52 0)
 			(effects
@@
 		)
 		(property "Description" "Generic connector, single row, 01x01, script generated (kicad-library-utils/schlib/autogen/connector/)"
+			(at 106.68 96.52 0)
+			(effects
+				(font
+					(size 1.27 1.27)
+				)
+				(hide yes)
+			)
+		)
+		(property "MPN" "S70-332002045R"
+			(at 106.68 96.52 0)
+			(effects
+				(font
+					(size 1.27 1.27)
+				)
+				(hide yes)
+			)
+		)
+		(property "Manufacturer" "Harwin"
 			(at 106.68 96.52 0)
 			(effects
@@
 			)
 		)
-		(property "Footprint" "footprints:S713145R"
+		(property "Footprint" "footprints:S70332002045R"
 			(at 106.68 74.93 0)
 			(effects
@@
 		)
 		(property "Description" "Generic connector, single row, 01x01, script generated (kicad-library-utils/schlib/autogen/connector/)"
+			(at 106.68 74.93 0)
+			(effects
+				(font
+					(size 1.27 1.27)
+				)
+				(hide yes)
+			)
+		)
+		(property "MPN" "S70-332002045R"
+			(at 106.68 74.93 0)
+			(effects
+				(font
+					(size 1.27 1.27)
+				)
+				(hide yes)
+			)
+		)
+		(property "Manufacturer" "Harwin"
 			(at 106.68 74.93 0)
 			(effects
@@
 				(path "/992fdb00-2079-4fab-820a-500481d674d7"
 					(reference "J4")
-					(unit 1)
-				)
-			)
-		)
-	)
-	(symbol
-		(lib_id "Mechanical:MountingHole")
-		(at 97.79 127 0)
-		(unit 1)
-		(exclude_from_sim yes)
-		(in_bom no)
-		(on_board yes)
-		(dnp no)
-		(fields_autoplaced yes)
-		(property "Reference" "H2"
-			(at 100.33 125.7299 0)
-			(effects
-				(font
-					(size 1.27 1.27)
-				)
-				(justify left)
-			)
-		)
-		(property "Value" "MountingHole"
-			(at 100.33 128.2699 0)
-			(effects
-				(font
-					(size 1.27 1.27)
-				)
-				(justify left)
-			)
-		)
-		(property "Footprint" "MountingHole:MountingHole_2.2mm_M2"
-			(at 97.79 127 0)
-			(effects
-				(font
-					(size 1.27 1.27)
-				)
-				(hide yes)
-			)
-		)
-		(property "Datasheet" "~"
-			(at 97.79 127 0)
-			(effects
-				(font
-					(size 1.27 1.27)
-				)
-				(hide yes)
-			)
-		)
-		(property "Description" "Mounting Hole without connection"
-			(at 97.79 127 0)
-			(effects
-				(font
-					(size 1.27 1.27)
-				)
-				(hide yes)
-			)
-		)
-		(instances
-			(project "nref-batterypack-backside"
-				(path "/992fdb00-2079-4fab-820a-500481d674d7"
-					(reference "H2")
 					(unit 1)
 				)
@@
 			)
 		)
+		(property "MPN" ""
+			(at 97.79 134.62 0)
+			(effects
+				(font
+					(size 1.27 1.27)
+				)
+				(hide yes)
+			)
+		)
+		(property "Manufacturer" ""
+			(at 97.79 134.62 0)
+			(effects
+				(font
+					(size 1.27 1.27)
+				)
+				(hide yes)
+			)
+		)
 		(instances
 			(project "nref-batterypack-backside"
@@
 			)
 		)
-		(property "Footprint" "Connector_JST:JST_SHL_SM02B-SHLS-TF_1x02-1MP_P1.00mm_Horizontal"
+		(property "Footprint" "Connector_JST:JST_SH_SM02B-SRSS-TB_1x02-1MP_P1.00mm_Horizontal"
 			(at 88.9 97.79 0)
 			(effects
@@
 		)
 		(property "Description" "Generic connector, single row, 01x02, script generated (kicad-library-utils/schlib/autogen/connector/)"
+			(at 88.9 97.79 0)
+			(effects
+				(font
+					(size 1.27 1.27)
+				)
+				(hide yes)
+			)
+		)
+		(property "MPN" "SM02B-SRSS-TB"
+			(at 88.9 97.79 0)
+			(effects
+				(font
+					(size 1.27 1.27)
+				)
+				(hide yes)
+			)
+		)
+		(property "Manufacturer" "JST"
 			(at 88.9 97.79 0)
 			(effects
@@
 			)
 		)
-		(property "Footprint" "footprints:S713145R"
+		(property "Footprint" "footprints:S174146R"
 			(at 106.68 85.09 0)
 			(effects
@@
 		)
 		(property "Description" "Generic connector, single row, 01x01, script generated (kicad-library-utils/schlib/autogen/connector/)"
+			(at 106.68 85.09 0)
+			(effects
+				(font
+					(size 1.27 1.27)
+				)
+				(hide yes)
+			)
+		)
+		(property "MPN" "S174146R"
+			(at 106.68 85.09 0)
+			(effects
+				(font
+					(size 1.27 1.27)
+				)
+				(hide yes)
+			)
+		)
+		(property "Manufacturer" "Harwin"
 			(at 106.68 85.09 0)
 			(effects
@@
 			)
 		)
-		(property "Footprint" "footprints:S713145R"
+		(property "Footprint" "footprints:S174146R"
 			(at 106.68 109.22 0)
 			(effects
@@
 		)
 		(property "Description" "Generic connector, single row, 01x01, script generated (kicad-library-utils/schlib/autogen/connector/)"
+			(at 106.68 109.22 0)
+			(effects
+				(font
+					(size 1.27 1.27)
+				)
+				(hide yes)
+			)
+		)
+		(property "MPN" "S174146R"
+			(at 106.68 109.22 0)
+			(effects
+				(font
+					(size 1.27 1.27)
+				)
+				(hide yes)
+			)
+		)
+		(property "Manufacturer" "Harwin"
 			(at 106.68 109.22 0)
 			(effects
@@
 			(at 97.79 120.65 0)
 			(effects
+				(font
+					(size 1.27 1.27)
+				)
+				(hide yes)
+			)
+		)
+		(property "MPN" ""
+			(at 97.79 120.65 0)
+			(effects
+				(font
+					(size 1.27 1.27)
+				)
+				(hide yes)
+			)
+		)
+		(property "Manufacturer" ""
+			(at 97.79 120.65 0)
+			(effects

Commit message: batterypack back/front: polishing for production
Parts:
- J1, J3: footprint footprints:S174146R -> footprints:Mill-Max_2036-X-57
- J2, J4: footprint footprints:S70332002045R -> footprints:MYOUNG_MY-FJ-115
Changed lines of the file:
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@@
 			)
 		)
-		(property "Footprint" "footprints:S70332002045R"
+		(property "Footprint" "footprints:MYOUNG_MY-FJ-115"
 			(at 106.68 96.52 0)
 			(effects
@@
 			)
 		)
-		(property "Footprint" "footprints:S70332002045R"
+		(property "Footprint" "footprints:MYOUNG_MY-FJ-115"
 			(at 106.68 74.93 0)
 			(effects
@@
 			)
 		)
-		(property "Footprint" "footprints:S174146R"
+		(property "Footprint" "footprints:Mill-Max_2036-X-57"
 			(at 106.68 85.09 0)
 			(effects
@@
 			)
 		)
-		(property "Footprint" "footprints:S174146R"
+		(property "Footprint" "footprints:Mill-Max_2036-X-57"
 			(at 106.68 109.22 0)
 			(effects
