File: nref-batterypack-v3/nref-batterypack-backside.kicad_sch (KiCad schematic)
At the start: 7 parts, among them J1 C1+, J2 C2-, J3 C3+, J4 C4-, J5 FRONT_CONN

Commit message: batterypack production updates
Parts:
- J1, J3: LCSC (none) -> C20777560; MPN S174146R -> 2036-3-57-15-00-00-03-0; Manufacturer Harwin -> Mill-Max
- J2, J4: LCSC (none) -> C5457098; MPN S70-332002045R -> MY-FJ-115II-R; Manufacturer Harwin -> MYOUNG
- J5: LCSC (none) -> C160402

Commit message: small schematic cleanups for book
Other:
- note added: "2-pin JST-SH cable to front side of pack"
- note added: "MNT Reform Next Battery Pack (Back Side)"
- company: (none) -> MNT Research GmbH, Copyright 2026
- title: (none) -> MNT Reform Next Battery Pack, Back Side
- moved on the sheet: H1, H3, J1, J2, J3, J4, J5
