File: nref-batterypack-v3/nref-batterypack.kicad_pcb (KiCad board)
At the start: 4 copper layers, 75 x 17 mm, 91 parts, among them J0 C1-, J1 C1-, J2 C2+, J3 C3-, J4 C4+, J5 PACK_CONN, J6 BACK_CONN, Q1 BC817, Q2 BC817, Q3 BC817, Q4 BC817, Q5 AO3401A, Q7 AO3401A, Q8 Q_Dual_NMOS_Picostar_CSD87501L, U1 BQ76922

Commit message: batterypack production updates
Parts:
- R1, R2, R3, R4: footprint Resistor_SMD:R_1210_3225Metric -> Resistor_SMD:R_1206_3216Metric
- moved TH4 0.95 mm to (166.9, 100.8)
- moved NT1 0.17 mm to (111.2, 100.2)
Routing:
- net /BATplus: track 18.0 -> 14.9 mm
- net VSS: track 48.8 -> 49.6 mm
- net Net-(Q1-C): track 1.81 -> 2.32 mm
- net GND: vias 102 -> 103
