File: nref-batterypack-v3/nref-batterypack.kicad_sch (KiCad schematic)
At the start: 90 parts, among them J0 C1-, J1 C1-, J2 C2+, J3 C3-, J4 C4+, J5 PACK_CONN, J6 BACK_CONN, Q1 BC817, Q2 BC817, Q3 BC817, Q4 BC817, Q5 AO3401A, Q7 AO3401A, Q8 Q_Dual_NMOS_Picostar_CSD87501L, U1 BQ76922

Commit message: batterypack production updates
Parts:
- D1: LCSC C95171 -> C22466375; MPN B140WS-7 -> B1040WS; Manufacturer Diodes -> R+O
- NT3, NT5: value ~ -> (none)
- R1, R2, R3, R4: footprint Resistor_SMD:R_1210_3225Metric -> Resistor_SMD:R_1206_3216Metric
