File: nref-trackpad-sensor/Trackpad_IQS9150.kicad_pcb (KiCad board)
At the start: 2 copper layers, 105.5 x 53.3 mm, 44 parts, among them CN1 FPC_6PIN, IC1 IQS9150-000QFR

Commit message: tpsensor: adjust exposed GND areas
Parts:
- H1: footprint footprints:nref-tpsensor-badge -> footprints:nref-tpsensor-badge-r2
Routing:
- net /Trackpad_IQS9150_1/GND: vias 62 -> 87

Commit message: trackpad pcb update for tight outline
Routing:
- net /Trackpad_IQS9150_1/COL18: track 121.1 -> 119.8 mm
- net /Trackpad_IQS9150_1/GND: vias 87 -> 85
