File: nref-wifi-m2/nref-wifi-m2.kicad_pcb (KiCad board)
At the start: 4 copper layers, 66 x 24 mm, 36 parts, among them J1 Bus_M.2_Socket_E, J2 Conn_01x20, U1 TPS62A04ABDRL, X1 ECS-327MVATX-2-CN-TR3

Commit message: wifi/bt board prod updates
Parts:
- L1: value 220nH XAL4020-221MEB -> 220nH 10A; footprint Inductor_SMD:L_Coilcraft_XAL4020-XXX -> EasyEDA:IND-SMD_L3.0-W3.0_FTC303020D
Routing:
- net GND: track 44.2 -> 48.2 mm, vias 78 -> 90
- net Net-(D2-K): track 12.4 -> 13.2 mm
